File: pcb/CS4272-CZZ_Breakout_Board.kicad_sch (KiCad schematic)
At the start: 65 parts, among them J1 Conn_01x14, J2 Conn_01x12, Q1 AO3401A, U1 CS4272, U2 SPX3819M5-L-3-3, Y1 24.576 MHz

Commit message: Update Ver 1
Parts:
- removed D1, D11, D12, D13, D14, D15, D16, D2, D3, D4, D5, D6, D7, D8, D9: D_TVS, Diode_SMD:D_0805_2012Metric, symbol Device:D_TVS
- C16, C17: value 40p -> 20p
- D1: renamed from D10; footprint Diode_SMD:D_0805_2012Metric -> Diode_SMD:D_SOD-323
- renumbered D17 to D2
Other:
- note added: "Transient Protection"
