File: pcb/multi-band-equalizer/analog_input_buffer.kicad_sch (KiCad schematic)
At the start: 16 parts, among them U7 NE5532

Commit message: pcb updates
Parts:
- renumbered C29 to C50, C30 to C51, C31 to C52, C32 to C53, C33 to C54, C34 to C55, C35 to C56, R35 to R50, R36 to R51, R37 to R52, R38 to R53, R39 to R54, R40 to R55, R41 to R56, R42 to R57

Commit message: sliding potentiometers
Parts:
- renumbered C50 to C52, C51 to C53, C52 to C54, C53 to C55, C54 to C56, C55 to C57, C56 to C58
Changed lines of the file:
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@@
 		(on_board yes)
 		(dnp no)
-		(property "Reference" "C52"
+		(property "Reference" "C54"
 			(at 256.54 83.058 90)
 			(effects
@@
 			(project ""
 				(path "/a5803ad9-a9e5-4a2c-ab35-f101ba189524/0c1d46b8-90f2-4124-b946-213bbd0984d2"
-					(reference "C52")
-					(unit 1)
-				)
-				(path "/a5803ad9-a9e5-4a2c-ab35-f101ba189524/af0974dd-017f-48f1-b391-cdf3f487ff20"
-					(reference "C59")
+					(reference "C54")
+					(unit 1)
+				)
+				(path "/a5803ad9-a9e5-4a2c-ab35-f101ba189524/af0974dd-017f-48f1-b391-cdf3f487ff20"
+					(reference "C61")
 					(unit 1)
 				)
@@
 		(dnp no)
 		(fields_autoplaced yes)
-		(property "Reference" "#PWR063"
+		(property "Reference" "#PWR064"
 			(at 80.01 123.19 0)
 			(effects
@@
 			(project ""
 				(path "/a5803ad9-a9e5-4a2c-ab35-f101ba189524/0c1d46b8-90f2-4124-b946-213bbd0984d2"
-					(reference "#PWR063")
-					(unit 1)
-				)
-				(path "/a5803ad9-a9e5-4a2c-ab35-f101ba189524/af0974dd-017f-48f1-b391-cdf3f487ff20"
-					(reference "#PWR068")
+					(reference "#PWR064")
+					(unit 1)
+				)
+				(path "/a5803ad9-a9e5-4a2c-ab35-f101ba189524/af0974dd-017f-48f1-b391-cdf3f487ff20"
+					(reference "#PWR069")
 					(unit 1)
 				)
@@
 		(dnp no)
 		(fields_autoplaced yes)
-		(property "Reference" "#PWR061"
+		(property "Reference" "#PWR062"
 			(at 240.03 116.84 0)
 			(effects
@@
 			(project ""
 				(path "/a5803ad9-a9e5-4a2c-ab35-f101ba189524/0c1d46b8-90f2-4124-b946-213bbd0984d2"
-					(reference "#PWR061")
-					(unit 1)
-				)
-				(path "/a5803ad9-a9e5-4a2c-ab35-f101ba189524/af0974dd-017f-48f1-b391-cdf3f487ff20"
-					(reference "#PWR066")
+					(reference "#PWR062")
+					(unit 1)
+				)
+				(path "/a5803ad9-a9e5-4a2c-ab35-f101ba189524/af0974dd-017f-48f1-b391-cdf3f487ff20"
+					(reference "#PWR067")
 					(unit 1)
 				)
@@
 		(dnp no)
 		(fields_autoplaced yes)
-		(property "Reference" "C54"
+		(property "Reference" "C56"
 			(at 83.82 110.4899 0)
 			(effects
@@
 			(project ""
 				(path "/a5803ad9-a9e5-4a2c-ab35-f101ba189524/0c1d46b8-90f2-4124-b946-213bbd0984d2"
-					(reference "C54")
-					(unit 1)
-				)
-				(path "/a5803ad9-a9e5-4a2c-ab35-f101ba189524/af0974dd-017f-48f1-b391-cdf3f487ff20"
-					(reference "C61")
+					(reference "C56")
+					(unit 1)
+				)
+				(path "/a5803ad9-a9e5-4a2c-ab35-f101ba189524/af0974dd-017f-48f1-b391-cdf3f487ff20"
+					(reference "C63")
 					(unit 1)
 				)
@@
 		(on_board yes)
 		(dnp no)
-		(property "Reference" "C55"
+		(property "Reference" "C57"
 			(at 148.59 111.252 90)
 			(effects
@@
 			(project ""
 				(path "/a5803ad9-a9e5-4a2c-ab35-f101ba189524/0c1d46b8-90f2-4124-b946-213bbd0984d2"
-					(reference "C55")
-					(unit 1)
-				)
-				(path "/a5803ad9-a9e5-4a2c-ab35-f101ba189524/af0974dd-017f-48f1-b391-cdf3f487ff20"
-					(reference "C62")
+					(reference "C57")
+					(unit 1)
+				)
+				(path "/a5803ad9-a9e5-4a2c-ab35-f101ba189524/af0974dd-017f-48f1-b391-cdf3f487ff20"
+					(reference "C64")
 					(unit 1)
 				)
@@
 		(dnp no)
 		(fields_autoplaced yes)
-		(property "Reference" "#PWR062"
+		(property "Reference" "#PWR063"
 			(at 46.99 119.38 0)
 			(effects
@@
 			(project ""
 				(path "/a5803ad9-a9e5-4a2c-ab35-f101ba189524/0c1d46b8-90f2-4124-b946-213bbd0984d2"
-					(reference "#PWR062")
-					(unit 1)
-				)
-				(path "/a5803ad9-a9e5-4a2c-ab35-f101ba189524/af0974dd-017f-48f1-b391-cdf3f487ff20"
-					(reference "#PWR067")
+					(reference "#PWR063")
+					(unit 1)
+				)
+				(path "/a5803ad9-a9e5-4a2c-ab35-f101ba189524/af0974dd-017f-48f1-b391-cdf3f487ff20"
+					(reference "#PWR068")
 					(unit 1)
 				)
@@
 		(dnp no)
 		(fields_autoplaced yes)
-		(property "Reference" "C53"
+		(property "Reference" "C55"
 			(at 196.85 107.9499 0)
 			(effects
@@
 			(project ""
 				(path "/a5803ad9-a9e5-4a2c-ab35-f101ba189524/0c1d46b8-90f2-4124-b946-213bbd0984d2"
-					(reference "C53")
-					(unit 1)
-				)
-				(path "/a5803ad9-a9e5-4a2c-ab35-f101ba189524/af0974dd-017f-48f1-b391-cdf3f487ff20"
-					(reference "C60")
+					(reference "C55")
+					(unit 1)
+				)
+				(path "/a5803ad9-a9e5-4a2c-ab35-f101ba189524/af0974dd-017f-48f1-b391-cdf3f487ff20"
+					(reference "C62")
 					(unit 1)
 				)
@@
 		(on_board yes)
 		(dnp no)
-		(property "Reference" "C51"
+		(property "Reference" "C53"
 			(at 79.883 77.47 90)
 			(effects
@@
 			(project ""
 				(path "/a5803ad9-a9e5-4a2c-ab35-f101ba189524/0c1d46b8-90f2-4124-b946-213bbd0984d2"
-					(reference "C51")
-					(unit 1)
-				)
-				(path "/a5803ad9-a9e5-4a2c-ab35-f101ba189524/af0974dd-017f-48f1-b391-cdf3f487ff20"
-					(reference "C58")
+					(reference "C53")
+					(unit 1)
+				)
+				(path "/a5803ad9-a9e5-4a2c-ab35-f101ba189524/af0974dd-017f-48f1-b391-cdf3f487ff20"
+					(reference "C60")
 					(unit 1)
 				)
@@
 		(dnp no)
 		(fields_autoplaced yes)
-		(property "Reference" "#PWR060"
+		(property "Reference" "#PWR061"
 			(at 262.89 100.33 0)
 			(effects
@@
 			(project ""
 				(path "/a5803ad9-a9e5-4a2c-ab35-f101ba189524/0c1d46b8-90f2-4124-b946-213bbd0984d2"
-					(reference "#PWR060")
-					(unit 1)
-				)
-				(path "/a5803ad9-a9e5-4a2c-ab35-f101ba189524/af0974dd-017f-48f1-b391-cdf3f487ff20"
-					(reference "#PWR065")
+					(reference "#PWR061")
+					(unit 1)
+				)
+				(path "/a5803ad9-a9e5-4a2c-ab35-f101ba189524/af0974dd-017f-48f1-b391-cdf3f487ff20"
+					(reference "#PWR066")
 					(unit 1)
 				)
@@
 		(on_board yes)
 		(dnp no)
-		(property "Reference" "C56"
+		(property "Reference" "C58"
 			(at 80.01 128.27 90)
 			(effects
@@
 			(project ""
 				(path "/a5803ad9-a9e5-4a2c-ab35-f101ba189524/0c1d46b8-90f2-4124-b946-213bbd0984d2"
-					(reference "C56")
-					(unit 1)
-				)
-				(path "/a5803ad9-a9e5-4a2c-ab35-f101ba189524/af0974dd-017f-48f1-b391-cdf3f487ff20"
-					(reference "C63")
+					(reference "C58")
+					(unit 1)
+				)
+				(path "/a5803ad9-a9e5-4a2c-ab35-f101ba189524/af0974dd-017f-48f1-b391-cdf3f487ff20"
+					(reference "C65")
 					(unit 1)
 				)
@@
 		(dnp no)
 		(fields_autoplaced yes)
-		(property "Reference" "#PWR059"
+		(property "Reference" "#PWR060"
 			(at 240.03 93.98 0)
 			(effects
@@
 			(project ""
 				(path "/a5803ad9-a9e5-4a2c-ab35-f101ba189524/0c1d46b8-90f2-4124-b946-213bbd0984d2"
-					(reference "#PWR059")
-					(unit 1)
-				)
-				(path "/a5803ad9-a9e5-4a2c-ab35-f101ba189524/af0974dd-017f-48f1-b391-cdf3f487ff20"
-					(reference "#PWR064")
+					(reference "#PWR060")
+					(unit 1)
+				)
+				(path "/a5803ad9-a9e5-4a2c-ab35-f101ba189524/af0974dd-017f-48f1-b391-cdf3f487ff20"
+					(reference "#PWR065")
 					(unit 1)
 				)
@@
 		(on_board yes)
 		(dnp no)
-		(property "Reference" "C50"
+		(property "Reference" "C52"
 			(at 148.59 60.452 90)
 			(effects
@@
 			(project ""
 				(path "/a5803ad9-a9e5-4a2c-ab35-f101ba189524/0c1d46b8-90f2-4124-b946-213bbd0984d2"
-					(reference "C50")
-					(unit 1)
-				)
-				(path "/a5803ad9-a9e5-4a2c-ab35-f101ba189524/af0974dd-017f-48f1-b391-cdf3f487ff20"
-					(reference "C57")
-					(unit 1)
-				)
+					(reference "C52")
+					(unit 1)
+				)
+				(path "/a5803ad9-a9e5-4a2c-ab35-f101ba189524/af0974dd-017f-48f1-b391-cdf3f487ff20"
+					(reference "C59")
+					(unit 1)
+				)

Commit message: Update pcb
Parts:
- renumbered C52 to C51, C53 to C52, C54 to C53, C55 to C54, C56 to C55, C57 to C56, C58 to C57, R50 to R49, R51 to R50, R52 to R51, R53 to R52, R54 to R53, R55 to R54, R56 to R55, R57 to R56

Commit message: Updated pcb and script
Parts:
- renumbered C51 to C54, C52 to C55, C53 to C56, C54 to C57, C55 to C58, C56 to C59, C57 to C60, R49 to R52, R50 to R53, R51 to R54, R52 to R55, R53 to R56, R54 to R57, R55 to R58, R56 to R59
Changed lines of the file:
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@@
 		(on_board yes)
 		(dnp no)
-		(property "Reference" "C53"
+		(property "Reference" "C56"
 			(at 256.54 83.058 90)
 			(effects
@@
 			(project ""
 				(path "/a5803ad9-a9e5-4a2c-ab35-f101ba189524/0c1d46b8-90f2-4124-b946-213bbd0984d2"
-					(reference "C53")
-					(unit 1)
-				)
-				(path "/a5803ad9-a9e5-4a2c-ab35-f101ba189524/af0974dd-017f-48f1-b391-cdf3f487ff20"
-					(reference "C60")
+					(reference "C56")
+					(unit 1)
+				)
+				(path "/a5803ad9-a9e5-4a2c-ab35-f101ba189524/af0974dd-017f-48f1-b391-cdf3f487ff20"
+					(reference "C63")
 					(unit 1)
 				)
@@
 		(dnp no)
 		(fields_autoplaced yes)
-		(property "Reference" "R52"
+		(property "Reference" "R55"
 			(at 104.14 91.4399 0)
 			(effects
@@
 			(project ""
 				(path "/a5803ad9-a9e5-4a2c-ab35-f101ba189524/0c1d46b8-90f2-4124-b946-213bbd0984d2"
-					(reference "R52")
-					(unit 1)
-				)
-				(path "/a5803ad9-a9e5-4a2c-ab35-f101ba189524/af0974dd-017f-48f1-b391-cdf3f487ff20"
-					(reference "R60")
+					(reference "R55")
+					(unit 1)
+				)
+				(path "/a5803ad9-a9e5-4a2c-ab35-f101ba189524/af0974dd-017f-48f1-b391-cdf3f487ff20"
+					(reference "R63")
 					(unit 1)
 				)
@@
 		(dnp no)
 		(fields_autoplaced yes)
-		(property "Reference" "R56"
+		(property "Reference" "R59"
 			(at 168.91 128.27 90)
 			(effects
@@
 			(project ""
 				(path "/a5803ad9-a9e5-4a2c-ab35-f101ba189524/0c1d46b8-90f2-4124-b946-213bbd0984d2"
-					(reference "R56")
-					(unit 1)
-				)
-				(path "/a5803ad9-a9e5-4a2c-ab35-f101ba189524/af0974dd-017f-48f1-b391-cdf3f487ff20"
-					(reference "R64")
+					(reference "R59")
+					(unit 1)
+				)
+				(path "/a5803ad9-a9e5-4a2c-ab35-f101ba189524/af0974dd-017f-48f1-b391-cdf3f487ff20"
+					(reference "R67")
 					(unit 1)
 				)
@@
 		(dnp no)
 		(fields_autoplaced yes)
-		(property "Reference" "C55"
+		(property "Reference" "C58"
 			(at 83.82 110.4899 0)
 			(effects
@@
 			(project ""
 				(path "/a5803ad9-a9e5-4a2c-ab35-f101ba189524/0c1d46b8-90f2-4124-b946-213bbd0984d2"
-					(reference "C55")
-					(unit 1)
-				)
-				(path "/a5803ad9-a9e5-4a2c-ab35-f101ba189524/af0974dd-017f-48f1-b391-cdf3f487ff20"
-					(reference "C62")
+					(reference "C58")
+					(unit 1)
+				)
+				(path "/a5803ad9-a9e5-4a2c-ab35-f101ba189524/af0974dd-017f-48f1-b391-cdf3f487ff20"
+					(reference "C65")
 					(unit 1)
 				)
@@
 		(on_board yes)
 		(dnp no)
-		(property "Reference" "C56"
+		(property "Reference" "C59"
 			(at 148.59 111.252 90)
 			(effects
@@
 			(project ""
 				(path "/a5803ad9-a9e5-4a2c-ab35-f101ba189524/0c1d46b8-90f2-4124-b946-213bbd0984d2"
-					(reference "C56")
-					(unit 1)
-				)
-				(path "/a5803ad9-a9e5-4a2c-ab35-f101ba189524/af0974dd-017f-48f1-b391-cdf3f487ff20"
-					(reference "C63")
+					(reference "C59")
+					(unit 1)
+				)
+				(path "/a5803ad9-a9e5-4a2c-ab35-f101ba189524/af0974dd-017f-48f1-b391-cdf3f487ff20"
+					(reference "C66")
 					(unit 1)
 				)
@@
 		(dnp no)
 		(fields_autoplaced yes)
-		(property "Reference" "R51"
+		(property "Reference" "R54"
 			(at 55.88 91.4399 0)
 			(effects
@@
 			(project ""
 				(path "/a5803ad9-a9e5-4a2c-ab35-f101ba189524/0c1d46b8-90f2-4124-b946-213bbd0984d2"
-					(reference "R51")
-					(unit 1)
-				)
-				(path "/a5803ad9-a9e5-4a2c-ab35-f101ba189524/af0974dd-017f-48f1-b391-cdf3f487ff20"
-					(reference "R59")
+					(reference "R54")
+					(unit 1)
+				)
+				(path "/a5803ad9-a9e5-4a2c-ab35-f101ba189524/af0974dd-017f-48f1-b391-cdf3f487ff20"
+					(reference "R62")
 					(unit 1)
 				)
@@
 		(dnp no)
 		(fields_autoplaced yes)
-		(property "Reference" "R50"
+		(property "Reference" "R53"
 			(at 168.91 77.47 90)
 			(effects
@@
 			(project ""
 				(path "/a5803ad9-a9e5-4a2c-ab35-f101ba189524/0c1d46b8-90f2-4124-b946-213bbd0984d2"
-					(reference "R50")
-					(unit 1)
-				)
-				(path "/a5803ad9-a9e5-4a2c-ab35-f101ba189524/af0974dd-017f-48f1-b391-cdf3f487ff20"
-					(reference "R58")
+					(reference "R53")
+					(unit 1)
+				)
+				(path "/a5803ad9-a9e5-4a2c-ab35-f101ba189524/af0974dd-017f-48f1-b391-cdf3f487ff20"
+					(reference "R61")
 					(unit 1)
 				)
@@
 		(dnp no)
 		(fields_autoplaced yes)
-		(property "Reference" "C54"
+		(property "Reference" "C57"
 			(at 196.85 107.9499 0)
 			(effects
@@
 			(project ""
 				(path "/a5803ad9-a9e5-4a2c-ab35-f101ba189524/0c1d46b8-90f2-4124-b946-213bbd0984d2"
-					(reference "C54")
-					(unit 1)
-				)
-				(path "/a5803ad9-a9e5-4a2c-ab35-f101ba189524/af0974dd-017f-48f1-b391-cdf3f487ff20"
-					(reference "C61")
+					(reference "C57")
+					(unit 1)
+				)
+				(path "/a5803ad9-a9e5-4a2c-ab35-f101ba189524/af0974dd-017f-48f1-b391-cdf3f487ff20"
+					(reference "C64")
 					(unit 1)
 				)
@@
 		(on_board yes)
 		(dnp no)
-		(property "Reference" "C52"
+		(property "Reference" "C55"
 			(at 79.883 77.47 90)
 			(effects
@@
 			(project ""
 				(path "/a5803ad9-a9e5-4a2c-ab35-f101ba189524/0c1d46b8-90f2-4124-b946-213bbd0984d2"
-					(reference "C52")
-					(unit 1)
-				)
-				(path "/a5803ad9-a9e5-4a2c-ab35-f101ba189524/af0974dd-017f-48f1-b391-cdf3f487ff20"
-					(reference "C59")
+					(reference "C55")
+					(unit 1)
+				)
+				(path "/a5803ad9-a9e5-4a2c-ab35-f101ba189524/af0974dd-017f-48f1-b391-cdf3f487ff20"
+					(reference "C62")
 					(unit 1)
 				)
@@
 		(on_board yes)
 		(dnp no)
-		(property "Reference" "C57"
+		(property "Reference" "C60"
 			(at 80.01 128.27 90)
 			(effects
@@
 			(project ""
 				(path "/a5803ad9-a9e5-4a2c-ab35-f101ba189524/0c1d46b8-90f2-4124-b946-213bbd0984d2"
-					(reference "C57")
-					(unit 1)
-				)
-				(path "/a5803ad9-a9e5-4a2c-ab35-f101ba189524/af0974dd-017f-48f1-b391-cdf3f487ff20"
-					(reference "C64")
+					(reference "C60")
+					(unit 1)
+				)
+				(path "/a5803ad9-a9e5-4a2c-ab35-f101ba189524/af0974dd-017f-48f1-b391-cdf3f487ff20"
+					(reference "C67")
 					(unit 1)
 				)
@@
 		(dnp no)
 		(fields_autoplaced yes)
-		(property "Reference" "R53"
+		(property "Reference" "R56"
 			(at 168.91 102.87 90)
 			(effects
@@
 			(project ""
 				(path "/a5803ad9-a9e5-4a2c-ab35-f101ba189524/0c1d46b8-90f2-4124-b946-213bbd0984d2"
-					(reference "R53")
-					(unit 1)
-				)
-				(path "/a5803ad9-a9e5-4a2c-ab35-f101ba189524/af0974dd-017f-48f1-b391-cdf3f487ff20"
-					(reference "R61")
+					(reference "R56")
+					(unit 1)
+				)
+				(path "/a5803ad9-a9e5-4a2c-ab35-f101ba189524/af0974dd-017f-48f1-b391-cdf3f487ff20"
+					(reference "R64")
 					(unit 1)
 				)
@@
 		(dnp no)
 		(fields_autoplaced yes)
-		(property "Reference" "R55"
+		(property "Reference" "R58"
 			(at 104.14 129.5399 0)
 			(effects
@@
 			(project ""
 				(path "/a5803ad9-a9e5-4a2c-ab35-f101ba189524/0c1d46b8-90f2-4124-b946-213bbd0984d2"
-					(reference "R55")
-					(unit 1)
-				)
-				(path "/a5803ad9-a9e5-4a2c-ab35-f101ba189524/af0974dd-017f-48f1-b391-cdf3f487ff20"
-					(reference "R63")
+					(reference "R58")
+					(unit 1)
+				)
+				(path "/a5803ad9-a9e5-4a2c-ab35-f101ba189524/af0974dd-017f-48f1-b391-cdf3f487ff20"
+					(reference "R66")
 					(unit 1)
 				)
@@
 		(dnp no)
 		(fields_autoplaced yes)
-		(property "Reference" "R54"
+		(property "Reference" "R57"
 			(at 55.88 129.5399 0)
 			(effects
@@
 			(project ""
 				(path "/a5803ad9-a9e5-4a2c-ab35-f101ba189524/0c1d46b8-90f2-4124-b946-213bbd0984d2"
-					(reference "R54")
-					(unit 1)
-				)
-				(path "/a5803ad9-a9e5-4a2c-ab35-f101ba189524/af0974dd-017f-48f1-b391-cdf3f487ff20"
-					(reference "R62")
+					(reference "R57")
+					(unit 1)
+				)
+				(path "/a5803ad9-a9e5-4a2c-ab35-f101ba189524/af0974dd-017f-48f1-b391-cdf3f487ff20"
+					(reference "R65")
 					(unit 1)
 				)
@@
 		(dnp no)
 		(fields_autoplaced yes)
-		(property "Reference" "R49"
+		(property "Reference" "R52"
 			(at 168.91 52.07 90)
 			(effects
@@
 			(project ""
 				(path "/a5803ad9-a9e5-4a2c-ab35-f101ba189524/0c1d46b8-90f2-4124-b946-213bbd0984d2"
-					(reference "R49")
-					(unit 1)
-				)
-				(path "/a5803ad9-a9e5-4a2c-ab35-f101ba189524/af0974dd-017f-48f1-b391-cdf3f487ff20"
-					(reference "R57")
+					(reference "R52")
+					(unit 1)
+				)
+				(path "/a5803ad9-a9e5-4a2c-ab35-f101ba189524/af0974dd-017f-48f1-b391-cdf3f487ff20"
+					(reference "R60")
 					(unit 1)
 				)
@@
 		(on_board yes)
 		(dnp no)
-		(property "Reference" "C51"
+		(property "Reference" "C54"
 			(at 148.59 60.452 90)
 			(effects
@@
 			(project ""
 				(path "/a5803ad9-a9e5-4a2c-ab35-f101ba189524/0c1d46b8-90f2-4124-b946-213bbd0984d2"
-					(reference "C51")
-					(unit 1)
-				)
-				(path "/a5803ad9-a9e5-4a2c-ab35-f101ba189524/af0974dd-017f-48f1-b391-cdf3f487ff20"
-					(reference "C58")
-					(unit 1)
-				)
+					(reference "C54")
+					(unit 1)
+				)
+				(path "/a5803ad9-a9e5-4a2c-ab35-f101ba189524/af0974dd-017f-48f1-b391-cdf3f487ff20"
+					(reference "C61")
+					(unit 1)
+				)
