File: pcb/multi-band-equalizer/analog_output_filter.kicad_sch (KiCad schematic)
At the start: 16 parts, among them U10 NE5532

Commit message: pcb updates
Parts:
- renumbered C50 to C71, C51 to C72, C52 to C73, C53 to C74, C54 to C75, C55 to C76, C56 to C77, R59 to R74, R60 to R75, R61 to R76, R62 to R77, R63 to R78, R64 to R79, R65 to R80, R66 to R81

Commit message: sliding potentiometers
Parts:
- renumbered C71 to C73, C72 to C74, C73 to C75, C74 to C76, C75 to C77, C76 to C78, C77 to C79
Changed lines of the file:
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@@
 		(dnp no)
 		(fields_autoplaced yes)
-		(property "Reference" "#PWR080"
+		(property "Reference" "#PWR081"
 			(at 187.96 121.92 0)
 			(effects
@@
 			(project "multi-band-equalizer"
 				(path "/a5803ad9-a9e5-4a2c-ab35-f101ba189524/0812df87-8f2b-4ce4-aa43-72c13c493f22"
-					(reference "#PWR080")
-					(unit 1)
-				)
-				(path "/a5803ad9-a9e5-4a2c-ab35-f101ba189524/acb16c71-e1a0-46fa-9ce3-74bbbdca6343"
-					(reference "#PWR073")
+					(reference "#PWR081")
+					(unit 1)
+				)
+				(path "/a5803ad9-a9e5-4a2c-ab35-f101ba189524/acb16c71-e1a0-46fa-9ce3-74bbbdca6343"
+					(reference "#PWR074")
 					(unit 1)
 				)
@@
 		(dnp no)
 		(fields_autoplaced yes)
-		(property "Reference" "#PWR076"
+		(property "Reference" "#PWR077"
 			(at 74.93 90.17 0)
 			(effects
@@
 			(project "multi-band-equalizer"
 				(path "/a5803ad9-a9e5-4a2c-ab35-f101ba189524/0812df87-8f2b-4ce4-aa43-72c13c493f22"
-					(reference "#PWR076")
-					(unit 1)
-				)
-				(path "/a5803ad9-a9e5-4a2c-ab35-f101ba189524/acb16c71-e1a0-46fa-9ce3-74bbbdca6343"
-					(reference "#PWR069")
+					(reference "#PWR077")
+					(unit 1)
+				)
+				(path "/a5803ad9-a9e5-4a2c-ab35-f101ba189524/acb16c71-e1a0-46fa-9ce3-74bbbdca6343"
+					(reference "#PWR070")
 					(unit 1)
 				)
@@
 		(on_board yes)
 		(dnp no)
-		(property "Reference" "C76"
+		(property "Reference" "C78"
 			(at 81.28 119.888 90)
 			(effects
@@
 			(project "multi-band-equalizer"
 				(path "/a5803ad9-a9e5-4a2c-ab35-f101ba189524/0812df87-8f2b-4ce4-aa43-72c13c493f22"
-					(reference "C76")
-					(unit 1)
-				)
-				(path "/a5803ad9-a9e5-4a2c-ab35-f101ba189524/acb16c71-e1a0-46fa-9ce3-74bbbdca6343"
-					(reference "C69")
+					(reference "C78")
+					(unit 1)
+				)
+				(path "/a5803ad9-a9e5-4a2c-ab35-f101ba189524/acb16c71-e1a0-46fa-9ce3-74bbbdca6343"
+					(reference "C71")
 					(unit 1)
 				)
@@
 		(on_board yes)
 		(dnp no)
-		(property "Reference" "C74"
+		(property "Reference" "C76"
 			(at 162.56 93.218 90)
 			(effects
@@
 			(project "multi-band-equalizer"
 				(path "/a5803ad9-a9e5-4a2c-ab35-f101ba189524/0812df87-8f2b-4ce4-aa43-72c13c493f22"
-					(reference "C74")
-					(unit 1)
-				)
-				(path "/a5803ad9-a9e5-4a2c-ab35-f101ba189524/acb16c71-e1a0-46fa-9ce3-74bbbdca6343"
-					(reference "C67")
+					(reference "C76")
+					(unit 1)
+				)
+				(path "/a5803ad9-a9e5-4a2c-ab35-f101ba189524/acb16c71-e1a0-46fa-9ce3-74bbbdca6343"
+					(reference "C69")
 					(unit 1)
 				)
@@
 		(on_board yes)
 		(dnp no)
-		(property "Reference" "C77"
+		(property "Reference" "C79"
 			(at 115.57 119.634 90)
 			(effects
@@
 			(project "multi-band-equalizer"
 				(path "/a5803ad9-a9e5-4a2c-ab35-f101ba189524/0812df87-8f2b-4ce4-aa43-72c13c493f22"
-					(reference "C77")
-					(unit 1)
-				)
-				(path "/a5803ad9-a9e5-4a2c-ab35-f101ba189524/acb16c71-e1a0-46fa-9ce3-74bbbdca6343"
-					(reference "C70")
+					(reference "C79")
+					(unit 1)
+				)
+				(path "/a5803ad9-a9e5-4a2c-ab35-f101ba189524/acb16c71-e1a0-46fa-9ce3-74bbbdca6343"
+					(reference "C72")
 					(unit 1)
 				)
@@
 		(dnp no)
 		(fields_autoplaced yes)
-		(property "Reference" "#PWR078"
+		(property "Reference" "#PWR079"
 			(at 246.38 95.25 0)
 			(effects
@@
 			(project "multi-band-equalizer"
 				(path "/a5803ad9-a9e5-4a2c-ab35-f101ba189524/0812df87-8f2b-4ce4-aa43-72c13c493f22"
-					(reference "#PWR078")
-					(unit 1)
-				)
-				(path "/a5803ad9-a9e5-4a2c-ab35-f101ba189524/acb16c71-e1a0-46fa-9ce3-74bbbdca6343"
-					(reference "#PWR071")
+					(reference "#PWR079")
+					(unit 1)
+				)
+				(path "/a5803ad9-a9e5-4a2c-ab35-f101ba189524/acb16c71-e1a0-46fa-9ce3-74bbbdca6343"
+					(reference "#PWR072")
 					(unit 1)
 				)
@@
 		(dnp no)
 		(fields_autoplaced yes)
-		(property "Reference" "#PWR082"
+		(property "Reference" "#PWR083"
 			(at 146.05 124.46 0)
 			(effects
@@
 			(project "multi-band-equalizer"
 				(path "/a5803ad9-a9e5-4a2c-ab35-f101ba189524/0812df87-8f2b-4ce4-aa43-72c13c493f22"
-					(reference "#PWR082")
-					(unit 1)
-				)
-				(path "/a5803ad9-a9e5-4a2c-ab35-f101ba189524/acb16c71-e1a0-46fa-9ce3-74bbbdca6343"
-					(reference "#PWR075")
+					(reference "#PWR083")
+					(unit 1)
+				)
+				(path "/a5803ad9-a9e5-4a2c-ab35-f101ba189524/acb16c71-e1a0-46fa-9ce3-74bbbdca6343"
+					(reference "#PWR076")
 					(unit 1)
 				)
@@
 		(on_board yes)
 		(dnp no)
-		(property "Reference" "C75"
+		(property "Reference" "C77"
 			(at 138.43 103.378 90)
 			(effects
@@
 			(project "multi-band-equalizer"
 				(path "/a5803ad9-a9e5-4a2c-ab35-f101ba189524/0812df87-8f2b-4ce4-aa43-72c13c493f22"
-					(reference "C75")
-					(unit 1)
-				)
-				(path "/a5803ad9-a9e5-4a2c-ab35-f101ba189524/acb16c71-e1a0-46fa-9ce3-74bbbdca6343"
-					(reference "C68")
+					(reference "C77")
+					(unit 1)
+				)
+				(path "/a5803ad9-a9e5-4a2c-ab35-f101ba189524/acb16c71-e1a0-46fa-9ce3-74bbbdca6343"
+					(reference "C70")
 					(unit 1)
 				)
@@
 		(on_board yes)
 		(dnp no)
-		(property "Reference" "C73"
+		(property "Reference" "C75"
 			(at 130.81 84.582 90)
 			(effects
@@
 			(project "multi-band-equalizer"
 				(path "/a5803ad9-a9e5-4a2c-ab35-f101ba189524/0812df87-8f2b-4ce4-aa43-72c13c493f22"
-					(reference "C73")
-					(unit 1)
-				)
-				(path "/a5803ad9-a9e5-4a2c-ab35-f101ba189524/acb16c71-e1a0-46fa-9ce3-74bbbdca6343"
-					(reference "C66")
+					(reference "C75")
+					(unit 1)
+				)
+				(path "/a5803ad9-a9e5-4a2c-ab35-f101ba189524/acb16c71-e1a0-46fa-9ce3-74bbbdca6343"
+					(reference "C68")
 					(unit 1)
 				)
@@
 		(dnp no)
 		(fields_autoplaced yes)
-		(property "Reference" "#PWR081"
+		(property "Reference" "#PWR082"
 			(at 74.93 123.19 0)
 			(effects
@@
 			(project "multi-band-equalizer"
 				(path "/a5803ad9-a9e5-4a2c-ab35-f101ba189524/0812df87-8f2b-4ce4-aa43-72c13c493f22"
-					(reference "#PWR081")
-					(unit 1)
-				)
-				(path "/a5803ad9-a9e5-4a2c-ab35-f101ba189524/acb16c71-e1a0-46fa-9ce3-74bbbdca6343"
-					(reference "#PWR074")
+					(reference "#PWR082")
+					(unit 1)
+				)
+				(path "/a5803ad9-a9e5-4a2c-ab35-f101ba189524/acb16c71-e1a0-46fa-9ce3-74bbbdca6343"
+					(reference "#PWR075")
 					(unit 1)
 				)
@@
 		(on_board yes)
 		(dnp no)
-		(property "Reference" "C72"
+		(property "Reference" "C74"
 			(at 240.03 77.978 90)
 			(effects
@@
 			(project "multi-band-equalizer"
 				(path "/a5803ad9-a9e5-4a2c-ab35-f101ba189524/0812df87-8f2b-4ce4-aa43-72c13c493f22"
-					(reference "C72")
-					(unit 1)
-				)
-				(path "/a5803ad9-a9e5-4a2c-ab35-f101ba189524/acb16c71-e1a0-46fa-9ce3-74bbbdca6343"
-					(reference "C65")
+					(reference "C74")
+					(unit 1)
+				)
+				(path "/a5803ad9-a9e5-4a2c-ab35-f101ba189524/acb16c71-e1a0-46fa-9ce3-74bbbdca6343"
+					(reference "C67")
 					(unit 1)
 				)
@@
 		(on_board yes)
 		(dnp no)
-		(property "Reference" "C71"
+		(property "Reference" "C73"
 			(at 81.28 73.66 90)
 			(effects
@@
 			(project "multi-band-equalizer"
 				(path "/a5803ad9-a9e5-4a2c-ab35-f101ba189524/0812df87-8f2b-4ce4-aa43-72c13c493f22"
-					(reference "C71")
-					(unit 1)
-				)
-				(path "/a5803ad9-a9e5-4a2c-ab35-f101ba189524/acb16c71-e1a0-46fa-9ce3-74bbbdca6343"
-					(reference "C64")
+					(reference "C73")
+					(unit 1)
+				)
+				(path "/a5803ad9-a9e5-4a2c-ab35-f101ba189524/acb16c71-e1a0-46fa-9ce3-74bbbdca6343"
+					(reference "C66")
 					(unit 1)
 				)
@@
 		(dnp no)
 		(fields_autoplaced yes)
-		(property "Reference" "#PWR077"
+		(property "Reference" "#PWR078"
 			(at 223.52 88.9 0)
 			(effects
@@
 			(project "multi-band-equalizer"
 				(path "/a5803ad9-a9e5-4a2c-ab35-f101ba189524/0812df87-8f2b-4ce4-aa43-72c13c493f22"
-					(reference "#PWR077")
-					(unit 1)
-				)
-				(path "/a5803ad9-a9e5-4a2c-ab35-f101ba189524/acb16c71-e1a0-46fa-9ce3-74bbbdca6343"
-					(reference "#PWR070")
+					(reference "#PWR078")
+					(unit 1)
+				)
+				(path "/a5803ad9-a9e5-4a2c-ab35-f101ba189524/acb16c71-e1a0-46fa-9ce3-74bbbdca6343"
+					(reference "#PWR071")
 					(unit 1)
 				)
@@
 		(dnp no)
 		(fields_autoplaced yes)
-		(property "Reference" "#PWR079"
+		(property "Reference" "#PWR080"
 			(at 223.52 111.76 0)
 			(effects
@@
 			(project "multi-band-equalizer"
 				(path "/a5803ad9-a9e5-4a2c-ab35-f101ba189524/0812df87-8f2b-4ce4-aa43-72c13c493f22"
-					(reference "#PWR079")
-					(unit 1)
-				)
-				(path "/a5803ad9-a9e5-4a2c-ab35-f101ba189524/acb16c71-e1a0-46fa-9ce3-74bbbdca6343"
-					(reference "#PWR072")
-					(unit 1)
-				)
+					(reference "#PWR080")
+					(unit 1)
+				)
+				(path "/a5803ad9-a9e5-4a2c-ab35-f101ba189524/acb16c71-e1a0-46fa-9ce3-74bbbdca6343"
+					(reference "#PWR073")
+					(unit 1)
+				)

Commit message: Update pcb
Parts:
- renumbered C73 to C72, C74 to C73, C75 to C74, C76 to C75, C77 to C76, C78 to C77, C79 to C78, R74 to R73, R75 to R74, R76 to R75, R77 to R76, R78 to R77, R79 to R78, R80 to R79, R81 to R80

Commit message: Updated pcb and script
Parts:
- renumbered C72 to C75, C73 to C76, C74 to C77, C75 to C78, C76 to C79, C77 to C80, C78 to C81, R73 to R76, R74 to R77, R75 to R78, R76 to R79, R77 to R80, R78 to R81, R79 to R82, R80 to R83
Changed lines of the file:
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@@
 		(on_board yes)
 		(dnp no)
-		(property "Reference" "R77"
+		(property "Reference" "R80"
 			(at 81.28 107.188 90)
 			(effects
@@
 			(project "multi-band-equalizer"
 				(path "/a5803ad9-a9e5-4a2c-ab35-f101ba189524/0812df87-8f2b-4ce4-aa43-72c13c493f22"
-					(reference "R77")
-					(unit 1)
-				)
-				(path "/a5803ad9-a9e5-4a2c-ab35-f101ba189524/acb16c71-e1a0-46fa-9ce3-74bbbdca6343"
-					(reference "R69")
+					(reference "R80")
+					(unit 1)
+				)
+				(path "/a5803ad9-a9e5-4a2c-ab35-f101ba189524/acb16c71-e1a0-46fa-9ce3-74bbbdca6343"
+					(reference "R72")
 					(unit 1)
 				)
@@
 		(dnp no)
 		(fields_autoplaced yes)
-		(property "Reference" "R79"
+		(property "Reference" "R82"
 			(at 190.5 107.9499 0)
 			(effects
@@
 			(project "multi-band-equalizer"
 				(path "/a5803ad9-a9e5-4a2c-ab35-f101ba189524/0812df87-8f2b-4ce4-aa43-72c13c493f22"
-					(reference "R79")
-					(unit 1)
-				)
-				(path "/a5803ad9-a9e5-4a2c-ab35-f101ba189524/acb16c71-e1a0-46fa-9ce3-74bbbdca6343"
-					(reference "R71")
+					(reference "R82")
+					(unit 1)
+				)
+				(path "/a5803ad9-a9e5-4a2c-ab35-f101ba189524/acb16c71-e1a0-46fa-9ce3-74bbbdca6343"
+					(reference "R74")
 					(unit 1)
 				)
@@
 		(on_board yes)
 		(dnp no)
-		(property "Reference" "C77"
+		(property "Reference" "C80"
 			(at 81.28 119.888 90)
 			(effects
@@
 			(project "multi-band-equalizer"
 				(path "/a5803ad9-a9e5-4a2c-ab35-f101ba189524/0812df87-8f2b-4ce4-aa43-72c13c493f22"
-					(reference "C77")
-					(unit 1)
-				)
-				(path "/a5803ad9-a9e5-4a2c-ab35-f101ba189524/acb16c71-e1a0-46fa-9ce3-74bbbdca6343"
-					(reference "C70")
+					(reference "C80")
+					(unit 1)
+				)
+				(path "/a5803ad9-a9e5-4a2c-ab35-f101ba189524/acb16c71-e1a0-46fa-9ce3-74bbbdca6343"
+					(reference "C73")
 					(unit 1)
 				)
@@
 		(on_board yes)
 		(dnp no)
-		(property "Reference" "C75"
+		(property "Reference" "C78"
 			(at 162.56 93.218 90)
 			(effects
@@
 			(project "multi-band-equalizer"
 				(path "/a5803ad9-a9e5-4a2c-ab35-f101ba189524/0812df87-8f2b-4ce4-aa43-72c13c493f22"
-					(reference "C75")
-					(unit 1)
-				)
-				(path "/a5803ad9-a9e5-4a2c-ab35-f101ba189524/acb16c71-e1a0-46fa-9ce3-74bbbdca6343"
-					(reference "C68")
+					(reference "C78")
+					(unit 1)
+				)
+				(path "/a5803ad9-a9e5-4a2c-ab35-f101ba189524/acb16c71-e1a0-46fa-9ce3-74bbbdca6343"
+					(reference "C71")
 					(unit 1)
 				)
@@
 		(on_board yes)
 		(dnp no)
-		(property "Reference" "C78"
+		(property "Reference" "C81"
 			(at 115.57 119.634 90)
 			(effects
@@
 			(project "multi-band-equalizer"
 				(path "/a5803ad9-a9e5-4a2c-ab35-f101ba189524/0812df87-8f2b-4ce4-aa43-72c13c493f22"
-					(reference "C78")
-					(unit 1)
-				)
-				(path "/a5803ad9-a9e5-4a2c-ab35-f101ba189524/acb16c71-e1a0-46fa-9ce3-74bbbdca6343"
-					(reference "C71")
+					(reference "C81")
+					(unit 1)
+				)
+				(path "/a5803ad9-a9e5-4a2c-ab35-f101ba189524/acb16c71-e1a0-46fa-9ce3-74bbbdca6343"
+					(reference "C74")
 					(unit 1)
 				)
@@
 		(on_board yes)
 		(dnp no)
-		(property "Reference" "R78"
+		(property "Reference" "R81"
 			(at 100.33 106.934 90)
 			(effects
@@
 			(project "multi-band-equalizer"
 				(path "/a5803ad9-a9e5-4a2c-ab35-f101ba189524/0812df87-8f2b-4ce4-aa43-72c13c493f22"
-					(reference "R78")
-					(unit 1)
-				)
-				(path "/a5803ad9-a9e5-4a2c-ab35-f101ba189524/acb16c71-e1a0-46fa-9ce3-74bbbdca6343"
-					(reference "R70")
+					(reference "R81")
+					(unit 1)
+				)
+				(path "/a5803ad9-a9e5-4a2c-ab35-f101ba189524/acb16c71-e1a0-46fa-9ce3-74bbbdca6343"
+					(reference "R73")
 					(unit 1)
 				)
@@
 		(dnp no)
 		(fields_autoplaced yes)
-		(property "Reference" "R73"
+		(property "Reference" "R76"
 			(at 114.3 76.2 90)
 			(effects
@@
 			(project "multi-band-equalizer"
 				(path "/a5803ad9-a9e5-4a2c-ab35-f101ba189524/0812df87-8f2b-4ce4-aa43-72c13c493f22"
-					(reference "R73")
-					(unit 1)
-				)
-				(path "/a5803ad9-a9e5-4a2c-ab35-f101ba189524/acb16c71-e1a0-46fa-9ce3-74bbbdca6343"
-					(reference "R65")
+					(reference "R76")
+					(unit 1)
+				)
+				(path "/a5803ad9-a9e5-4a2c-ab35-f101ba189524/acb16c71-e1a0-46fa-9ce3-74bbbdca6343"
+					(reference "R68")
 					(unit 1)
 				)
@@
 		(dnp no)
 		(fields_autoplaced yes)
-		(property "Reference" "R74"
+		(property "Reference" "R77"
 			(at 81.28 92.71 90)
 			(effects
@@
 			(project "multi-band-equalizer"
 				(path "/a5803ad9-a9e5-4a2c-ab35-f101ba189524/0812df87-8f2b-4ce4-aa43-72c13c493f22"
-					(reference "R74")
-					(unit 1)
-				)
-				(path "/a5803ad9-a9e5-4a2c-ab35-f101ba189524/acb16c71-e1a0-46fa-9ce3-74bbbdca6343"
-					(reference "R66")
+					(reference "R77")
+					(unit 1)
+				)
+				(path "/a5803ad9-a9e5-4a2c-ab35-f101ba189524/acb16c71-e1a0-46fa-9ce3-74bbbdca6343"
+					(reference "R69")
 					(unit 1)
 				)
@@
 		(on_board yes)
 		(dnp no)
-		(property "Reference" "C76"
+		(property "Reference" "C79"
 			(at 138.43 103.378 90)
 			(effects
@@
 			(project "multi-band-equalizer"
 				(path "/a5803ad9-a9e5-4a2c-ab35-f101ba189524/0812df87-8f2b-4ce4-aa43-72c13c493f22"
-					(reference "C76")
-					(unit 1)
-				)
-				(path "/a5803ad9-a9e5-4a2c-ab35-f101ba189524/acb16c71-e1a0-46fa-9ce3-74bbbdca6343"
-					(reference "C69")
+					(reference "C79")
+					(unit 1)
+				)
+				(path "/a5803ad9-a9e5-4a2c-ab35-f101ba189524/acb16c71-e1a0-46fa-9ce3-74bbbdca6343"
+					(reference "C72")
 					(unit 1)
 				)
@@
 		(on_board yes)
 		(dnp no)
-		(property "Reference" "C74"
+		(property "Reference" "C77"
 			(at 130.81 84.582 90)
 			(effects
@@
 			(project "multi-band-equalizer"
 				(path "/a5803ad9-a9e5-4a2c-ab35-f101ba189524/0812df87-8f2b-4ce4-aa43-72c13c493f22"
-					(reference "C74")
-					(unit 1)
-				)
-				(path "/a5803ad9-a9e5-4a2c-ab35-f101ba189524/acb16c71-e1a0-46fa-9ce3-74bbbdca6343"
-					(reference "C67")
+					(reference "C77")
+					(unit 1)
+				)
+				(path "/a5803ad9-a9e5-4a2c-ab35-f101ba189524/acb16c71-e1a0-46fa-9ce3-74bbbdca6343"
+					(reference "C70")
 					(unit 1)
 				)
@@
 		(dnp no)
 		(fields_autoplaced yes)
-		(property "Reference" "R75"
+		(property "Reference" "R78"
 			(at 100.33 92.71 90)
 			(effects
@@
 			(project "multi-band-equalizer"
 				(path "/a5803ad9-a9e5-4a2c-ab35-f101ba189524/0812df87-8f2b-4ce4-aa43-72c13c493f22"
-					(reference "R75")
-					(unit 1)
-				)
-				(path "/a5803ad9-a9e5-4a2c-ab35-f101ba189524/acb16c71-e1a0-46fa-9ce3-74bbbdca6343"
-					(reference "R67")
+					(reference "R78")
+					(unit 1)
+				)
+				(path "/a5803ad9-a9e5-4a2c-ab35-f101ba189524/acb16c71-e1a0-46fa-9ce3-74bbbdca6343"
+					(reference "R70")
 					(unit 1)
 				)
@@
 		(dnp no)
 		(fields_autoplaced yes)
-		(property "Reference" "R76"
+		(property "Reference" "R79"
 			(at 176.53 95.25 90)
 			(effects
@@
 			(project "multi-band-equalizer"
 				(path "/a5803ad9-a9e5-4a2c-ab35-f101ba189524/0812df87-8f2b-4ce4-aa43-72c13c493f22"
-					(reference "R76")
-					(unit 1)
-				)
-				(path "/a5803ad9-a9e5-4a2c-ab35-f101ba189524/acb16c71-e1a0-46fa-9ce3-74bbbdca6343"
-					(reference "R68")
+					(reference "R79")
+					(unit 1)
+				)
+				(path "/a5803ad9-a9e5-4a2c-ab35-f101ba189524/acb16c71-e1a0-46fa-9ce3-74bbbdca6343"
+					(reference "R71")
 					(unit 1)
 				)
@@
 		(on_board yes)
 		(dnp no)
-		(property "Reference" "R80"
+		(property "Reference" "R83"
 			(at 100.33 118.364 90)
 			(effects
@@
 			(project "multi-band-equalizer"
 				(path "/a5803ad9-a9e5-4a2c-ab35-f101ba189524/0812df87-8f2b-4ce4-aa43-72c13c493f22"
-					(reference "R80")
-					(unit 1)
-				)
-				(path "/a5803ad9-a9e5-4a2c-ab35-f101ba189524/acb16c71-e1a0-46fa-9ce3-74bbbdca6343"
-					(reference "R72")
+					(reference "R83")
+					(unit 1)
+				)
+				(path "/a5803ad9-a9e5-4a2c-ab35-f101ba189524/acb16c71-e1a0-46fa-9ce3-74bbbdca6343"
+					(reference "R75")
 					(unit 1)
 				)
@@
 		(on_board yes)
 		(dnp no)
-		(property "Reference" "C73"
+		(property "Reference" "C76"
 			(at 240.03 77.978 90)
 			(effects
@@
 			(project "multi-band-equalizer"
 				(path "/a5803ad9-a9e5-4a2c-ab35-f101ba189524/0812df87-8f2b-4ce4-aa43-72c13c493f22"
-					(reference "C73")
-					(unit 1)
-				)
-				(path "/a5803ad9-a9e5-4a2c-ab35-f101ba189524/acb16c71-e1a0-46fa-9ce3-74bbbdca6343"
-					(reference "C66")
+					(reference "C76")
+					(unit 1)
+				)
+				(path "/a5803ad9-a9e5-4a2c-ab35-f101ba189524/acb16c71-e1a0-46fa-9ce3-74bbbdca6343"
+					(reference "C69")
 					(unit 1)
 				)
@@
 		(on_board yes)
 		(dnp no)
-		(property "Reference" "C72"
+		(property "Reference" "C75"
 			(at 81.28 73.66 90)
 			(effects
@@
 			(project "multi-band-equalizer"
 				(path "/a5803ad9-a9e5-4a2c-ab35-f101ba189524/0812df87-8f2b-4ce4-aa43-72c13c493f22"
-					(reference "C72")
-					(unit 1)
-				)
-				(path "/a5803ad9-a9e5-4a2c-ab35-f101ba189524/acb16c71-e1a0-46fa-9ce3-74bbbdca6343"
-					(reference "C65")
-					(unit 1)
-				)
+					(reference "C75")
+					(unit 1)
+				)
+				(path "/a5803ad9-a9e5-4a2c-ab35-f101ba189524/acb16c71-e1a0-46fa-9ce3-74bbbdca6343"
+					(reference "C68")
+					(unit 1)
+				)
