File: pcb/multi-band-equalizer/single_to_differential.kicad_sch (KiCad schematic)
At the start: 16 parts, among them U6 NE5532

Commit message: pcb updates
Parts:
- renumbered C25 to C46, C26 to C47, C27 to C48, C28 to C49, R24 to R39, R25 to R40, R26 to R41, R27 to R42, R28 to R43, R29 to R44, R30 to R45, R31 to R46, R32 to R47, R33 to R48, R34 to R49

Commit message: sliding potentiometers
Parts:
- renumbered C46 to C48, C47 to C49, C48 to C50, C49 to C51
Changed lines of the file:
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@@
 		(dnp no)
 		(fields_autoplaced yes)
-		(property "Reference" "#PWR049"
+		(property "Reference" "#PWR050"
 			(at 130.81 50.8 0)
 			(effects
@@
 			(project "multi-band-equalizer"
 				(path "/a5803ad9-a9e5-4a2c-ab35-f101ba189524/45ab872a-c810-43fb-b03d-ad8b0d23cb6b"
-					(reference "#PWR049")
-					(unit 1)
-				)
-				(path "/a5803ad9-a9e5-4a2c-ab35-f101ba189524/838129ab-a80a-454e-bedd-d4d19cd21db9"
-					(reference "#PWR039")
+					(reference "#PWR050")
+					(unit 1)
+				)
+				(path "/a5803ad9-a9e5-4a2c-ab35-f101ba189524/838129ab-a80a-454e-bedd-d4d19cd21db9"
+					(reference "#PWR040")
 					(unit 1)
 				)
@@
 		(dnp no)
 		(fields_autoplaced yes)
-		(property "Reference" "#PWR057"
+		(property "Reference" "#PWR058"
 			(at 195.58 105.41 0)
 			(effects
@@
 			(project "multi-band-equalizer"
 				(path "/a5803ad9-a9e5-4a2c-ab35-f101ba189524/45ab872a-c810-43fb-b03d-ad8b0d23cb6b"
-					(reference "#PWR057")
-					(unit 1)
-				)
-				(path "/a5803ad9-a9e5-4a2c-ab35-f101ba189524/838129ab-a80a-454e-bedd-d4d19cd21db9"
-					(reference "#PWR047")
+					(reference "#PWR058")
+					(unit 1)
+				)
+				(path "/a5803ad9-a9e5-4a2c-ab35-f101ba189524/838129ab-a80a-454e-bedd-d4d19cd21db9"
+					(reference "#PWR048")
 					(unit 1)
 				)
@@
 		(dnp no)
 		(fields_autoplaced yes)
-		(property "Reference" "#PWR052"
+		(property "Reference" "#PWR053"
 			(at 158.75 69.85 0)
 			(effects
@@
 			(project "multi-band-equalizer"
 				(path "/a5803ad9-a9e5-4a2c-ab35-f101ba189524/45ab872a-c810-43fb-b03d-ad8b0d23cb6b"
-					(reference "#PWR052")
-					(unit 1)
-				)
-				(path "/a5803ad9-a9e5-4a2c-ab35-f101ba189524/838129ab-a80a-454e-bedd-d4d19cd21db9"
-					(reference "#PWR042")
+					(reference "#PWR053")
+					(unit 1)
+				)
+				(path "/a5803ad9-a9e5-4a2c-ab35-f101ba189524/838129ab-a80a-454e-bedd-d4d19cd21db9"
+					(reference "#PWR043")
 					(unit 1)
 				)
@@
 		(dnp no)
 		(fields_autoplaced yes)
-		(property "Reference" "#PWR053"
+		(property "Reference" "#PWR054"
 			(at 233.68 80.01 0)
 			(effects
@@
 			(project "multi-band-equalizer"
 				(path "/a5803ad9-a9e5-4a2c-ab35-f101ba189524/45ab872a-c810-43fb-b03d-ad8b0d23cb6b"
-					(reference "#PWR053")
-					(unit 1)
-				)
-				(path "/a5803ad9-a9e5-4a2c-ab35-f101ba189524/838129ab-a80a-454e-bedd-d4d19cd21db9"
-					(reference "#PWR043")
+					(reference "#PWR054")
+					(unit 1)
+				)
+				(path "/a5803ad9-a9e5-4a2c-ab35-f101ba189524/838129ab-a80a-454e-bedd-d4d19cd21db9"
+					(reference "#PWR044")
 					(unit 1)
 				)
@@
 		(dnp no)
 		(fields_autoplaced yes)
-		(property "Reference" "#PWR054"
+		(property "Reference" "#PWR055"
 			(at 66.04 102.87 0)
 			(effects
@@
 			(project "multi-band-equalizer"
 				(path "/a5803ad9-a9e5-4a2c-ab35-f101ba189524/45ab872a-c810-43fb-b03d-ad8b0d23cb6b"
-					(reference "#PWR054")
-					(unit 1)
-				)
-				(path "/a5803ad9-a9e5-4a2c-ab35-f101ba189524/838129ab-a80a-454e-bedd-d4d19cd21db9"
-					(reference "#PWR044")
+					(reference "#PWR055")
+					(unit 1)
+				)
+				(path "/a5803ad9-a9e5-4a2c-ab35-f101ba189524/838129ab-a80a-454e-bedd-d4d19cd21db9"
+					(reference "#PWR045")
 					(unit 1)
 				)
@@
 		(dnp no)
 		(fields_autoplaced yes)
-		(property "Reference" "#PWR058"
+		(property "Reference" "#PWR059"
 			(at 195.58 144.78 0)
 			(effects
@@
 			(project "multi-band-equalizer"
 				(path "/a5803ad9-a9e5-4a2c-ab35-f101ba189524/45ab872a-c810-43fb-b03d-ad8b0d23cb6b"
-					(reference "#PWR058")
-					(unit 1)
-				)
-				(path "/a5803ad9-a9e5-4a2c-ab35-f101ba189524/838129ab-a80a-454e-bedd-d4d19cd21db9"
-					(reference "#PWR048")
+					(reference "#PWR059")
+					(unit 1)
+				)
+				(path "/a5803ad9-a9e5-4a2c-ab35-f101ba189524/838129ab-a80a-454e-bedd-d4d19cd21db9"
+					(reference "#PWR049")
 					(unit 1)
 				)
@@
 		(dnp no)
 		(fields_autoplaced yes)
-		(property "Reference" "C47"
+		(property "Reference" "C49"
 			(at 119.38 73.66 90)
 			(effects
@@
 			(project "multi-band-equalizer"
 				(path "/a5803ad9-a9e5-4a2c-ab35-f101ba189524/45ab872a-c810-43fb-b03d-ad8b0d23cb6b"
-					(reference "C47")
-					(unit 1)
-				)
-				(path "/a5803ad9-a9e5-4a2c-ab35-f101ba189524/838129ab-a80a-454e-bedd-d4d19cd21db9"
-					(reference "C43")
+					(reference "C49")
+					(unit 1)
+				)
+				(path "/a5803ad9-a9e5-4a2c-ab35-f101ba189524/838129ab-a80a-454e-bedd-d4d19cd21db9"
+					(reference "C45")
 					(unit 1)
 				)
@@
 		(dnp no)
 		(fields_autoplaced yes)
-		(property "Reference" "#PWR050"
+		(property "Reference" "#PWR051"
 			(at 233.68 57.15 0)
 			(effects
@@
 			(project "multi-band-equalizer"
 				(path "/a5803ad9-a9e5-4a2c-ab35-f101ba189524/45ab872a-c810-43fb-b03d-ad8b0d23cb6b"
-					(reference "#PWR050")
-					(unit 1)
-				)
-				(path "/a5803ad9-a9e5-4a2c-ab35-f101ba189524/838129ab-a80a-454e-bedd-d4d19cd21db9"
-					(reference "#PWR040")
+					(reference "#PWR051")
+					(unit 1)
+				)
+				(path "/a5803ad9-a9e5-4a2c-ab35-f101ba189524/838129ab-a80a-454e-bedd-d4d19cd21db9"
+					(reference "#PWR041")
 					(unit 1)
 				)
@@
 		(dnp no)
 		(fields_autoplaced yes)
-		(property "Reference" "#PWR056"
+		(property "Reference" "#PWR057"
 			(at 105.41 102.87 0)
 			(effects
@@
 			(project "multi-band-equalizer"
 				(path "/a5803ad9-a9e5-4a2c-ab35-f101ba189524/45ab872a-c810-43fb-b03d-ad8b0d23cb6b"
-					(reference "#PWR056")
-					(unit 1)
-				)
-				(path "/a5803ad9-a9e5-4a2c-ab35-f101ba189524/838129ab-a80a-454e-bedd-d4d19cd21db9"
-					(reference "#PWR046")
+					(reference "#PWR057")
+					(unit 1)
+				)
+				(path "/a5803ad9-a9e5-4a2c-ab35-f101ba189524/838129ab-a80a-454e-bedd-d4d19cd21db9"
+					(reference "#PWR047")
 					(unit 1)
 				)
@@
 		(dnp no)
 		(fields_autoplaced yes)
-		(property "Reference" "#PWR051"
+		(property "Reference" "#PWR052"
 			(at 256.54 63.5 0)
 			(effects
@@
 			(project "multi-band-equalizer"
 				(path "/a5803ad9-a9e5-4a2c-ab35-f101ba189524/45ab872a-c810-43fb-b03d-ad8b0d23cb6b"
-					(reference "#PWR051")
-					(unit 1)
-				)
-				(path "/a5803ad9-a9e5-4a2c-ab35-f101ba189524/838129ab-a80a-454e-bedd-d4d19cd21db9"
-					(reference "#PWR041")
+					(reference "#PWR052")
+					(unit 1)
+				)
+				(path "/a5803ad9-a9e5-4a2c-ab35-f101ba189524/838129ab-a80a-454e-bedd-d4d19cd21db9"
+					(reference "#PWR042")
 					(unit 1)
 				)
@@
 		(dnp no)
 		(fields_autoplaced yes)
-		(property "Reference" "#PWR055"
+		(property "Reference" "#PWR056"
 			(at 85.09 102.87 0)
 			(effects
@@
 			(project "multi-band-equalizer"
 				(path "/a5803ad9-a9e5-4a2c-ab35-f101ba189524/45ab872a-c810-43fb-b03d-ad8b0d23cb6b"
-					(reference "#PWR055")
-					(unit 1)
-				)
-				(path "/a5803ad9-a9e5-4a2c-ab35-f101ba189524/838129ab-a80a-454e-bedd-d4d19cd21db9"
-					(reference "#PWR045")
+					(reference "#PWR056")
+					(unit 1)
+				)
+				(path "/a5803ad9-a9e5-4a2c-ab35-f101ba189524/838129ab-a80a-454e-bedd-d4d19cd21db9"
+					(reference "#PWR046")
 					(unit 1)
 				)
@@
 		(on_board yes)
 		(dnp no)
-		(property "Reference" "C49"
+		(property "Reference" "C51"
 			(at 168.91 150.622 90)
 			(effects
@@
 			(project "multi-band-equalizer"
 				(path "/a5803ad9-a9e5-4a2c-ab35-f101ba189524/45ab872a-c810-43fb-b03d-ad8b0d23cb6b"
-					(reference "C49")
-					(unit 1)
-				)
-				(path "/a5803ad9-a9e5-4a2c-ab35-f101ba189524/838129ab-a80a-454e-bedd-d4d19cd21db9"
-					(reference "C45")
+					(reference "C51")
+					(unit 1)
+				)
+				(path "/a5803ad9-a9e5-4a2c-ab35-f101ba189524/838129ab-a80a-454e-bedd-d4d19cd21db9"
+					(reference "C47")
 					(unit 1)
 				)
@@
 		(dnp no)
 		(fields_autoplaced yes)
-		(property "Reference" "C46"
+		(property "Reference" "C48"
 			(at 250.19 46.99 90)
 			(effects
@@
 			(project "multi-band-equalizer"
 				(path "/a5803ad9-a9e5-4a2c-ab35-f101ba189524/45ab872a-c810-43fb-b03d-ad8b0d23cb6b"
-					(reference "C46")
-					(unit 1)
-				)
-				(path "/a5803ad9-a9e5-4a2c-ab35-f101ba189524/838129ab-a80a-454e-bedd-d4d19cd21db9"
-					(reference "C42")
+					(reference "C48")
+					(unit 1)
+				)
+				(path "/a5803ad9-a9e5-4a2c-ab35-f101ba189524/838129ab-a80a-454e-bedd-d4d19cd21db9"
+					(reference "C44")
 					(unit 1)
 				)
@@
 		(dnp no)
 		(fields_autoplaced yes)
-		(property "Reference" "C48"
+		(property "Reference" "C50"
 			(at 88.9 87.6299 0)
 			(effects
@@
 			(project "multi-band-equalizer"
 				(path "/a5803ad9-a9e5-4a2c-ab35-f101ba189524/45ab872a-c810-43fb-b03d-ad8b0d23cb6b"
-					(reference "C48")
-					(unit 1)
-				)
-				(path "/a5803ad9-a9e5-4a2c-ab35-f101ba189524/838129ab-a80a-454e-bedd-d4d19cd21db9"
-					(reference "C44")
-					(unit 1)
-				)
+					(reference "C50")
+					(unit 1)
+				)
+				(path "/a5803ad9-a9e5-4a2c-ab35-f101ba189524/838129ab-a80a-454e-bedd-d4d19cd21db9"
+					(reference "C46")
+					(unit 1)
+				)

Commit message: Update pcb
Parts:
- renumbered C48 to C47, C49 to C48, C50 to C49, C51 to C50, R39 to R38, R40 to R39, R41 to R40, R42 to R41, R43 to R42, R44 to R43, R45 to R44, R46 to R45, R47 to R46, R48 to R47, R49 to R48

Commit message: Updated pcb and script
Parts:
- renumbered C47 to C50, C48 to C51, C49 to C52, C50 to C53, R38 to R41, R39 to R42, R40 to R43, R41 to R44, R42 to R45, R43 to R46, R44 to R47, R45 to R48, R46 to R49, R47 to R50, R48 to R51
Changed lines of the file:
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@@
 		(dnp no)
 		(fields_autoplaced yes)
-		(property "Reference" "R44"
+		(property "Reference" "R47"
 			(at 198.12 91.4399 0)
 			(effects
@@
 			(project "multi-band-equalizer"
 				(path "/a5803ad9-a9e5-4a2c-ab35-f101ba189524/45ab872a-c810-43fb-b03d-ad8b0d23cb6b"
-					(reference "R44")
-					(unit 1)
-				)
-				(path "/a5803ad9-a9e5-4a2c-ab35-f101ba189524/838129ab-a80a-454e-bedd-d4d19cd21db9"
-					(reference "R33")
+					(reference "R47")
+					(unit 1)
+				)
+				(path "/a5803ad9-a9e5-4a2c-ab35-f101ba189524/838129ab-a80a-454e-bedd-d4d19cd21db9"
+					(reference "R36")
 					(unit 1)
 				)
@@
 		(dnp no)
 		(fields_autoplaced yes)
-		(property "Reference" "R40"
+		(property "Reference" "R43"
 			(at 133.35 72.3899 0)
 			(effects
@@
 			(project "multi-band-equalizer"
 				(path "/a5803ad9-a9e5-4a2c-ab35-f101ba189524/45ab872a-c810-43fb-b03d-ad8b0d23cb6b"
-					(reference "R40")
-					(unit 1)
-				)
-				(path "/a5803ad9-a9e5-4a2c-ab35-f101ba189524/838129ab-a80a-454e-bedd-d4d19cd21db9"
-					(reference "R29")
+					(reference "R43")
+					(unit 1)
+				)
+				(path "/a5803ad9-a9e5-4a2c-ab35-f101ba189524/838129ab-a80a-454e-bedd-d4d19cd21db9"
+					(reference "R32")
 					(unit 1)
 				)
@@
 		(dnp no)
 		(fields_autoplaced yes)
-		(property "Reference" "R46"
+		(property "Reference" "R49"
 			(at 152.4 115.5699 0)
 			(effects
@@
 			(project "multi-band-equalizer"
 				(path "/a5803ad9-a9e5-4a2c-ab35-f101ba189524/45ab872a-c810-43fb-b03d-ad8b0d23cb6b"
-					(reference "R46")
-					(unit 1)
-				)
-				(path "/a5803ad9-a9e5-4a2c-ab35-f101ba189524/838129ab-a80a-454e-bedd-d4d19cd21db9"
-					(reference "R35")
+					(reference "R49")
+					(unit 1)
+				)
+				(path "/a5803ad9-a9e5-4a2c-ab35-f101ba189524/838129ab-a80a-454e-bedd-d4d19cd21db9"
+					(reference "R38")
 					(unit 1)
 				)
@@
 		(dnp no)
 		(fields_autoplaced yes)
-		(property "Reference" "R47"
+		(property "Reference" "R50"
 			(at 198.12 130.8099 0)
 			(effects
@@
 			(project "multi-band-equalizer"
 				(path "/a5803ad9-a9e5-4a2c-ab35-f101ba189524/45ab872a-c810-43fb-b03d-ad8b0d23cb6b"
-					(reference "R47")
-					(unit 1)
-				)
-				(path "/a5803ad9-a9e5-4a2c-ab35-f101ba189524/838129ab-a80a-454e-bedd-d4d19cd21db9"
-					(reference "R36")
+					(reference "R50")
+					(unit 1)
+				)
+				(path "/a5803ad9-a9e5-4a2c-ab35-f101ba189524/838129ab-a80a-454e-bedd-d4d19cd21db9"
+					(reference "R39")
 					(unit 1)
 				)
@@
 		(dnp no)
 		(fields_autoplaced yes)
-		(property "Reference" "R41"
+		(property "Reference" "R44"
 			(at 55.88 74.93 90)
 			(effects
@@
 			(project "multi-band-equalizer"
 				(path "/a5803ad9-a9e5-4a2c-ab35-f101ba189524/45ab872a-c810-43fb-b03d-ad8b0d23cb6b"
-					(reference "R41")
-					(unit 1)
-				)
-				(path "/a5803ad9-a9e5-4a2c-ab35-f101ba189524/838129ab-a80a-454e-bedd-d4d19cd21db9"
-					(reference "R30")
+					(reference "R44")
+					(unit 1)
+				)
+				(path "/a5803ad9-a9e5-4a2c-ab35-f101ba189524/838129ab-a80a-454e-bedd-d4d19cd21db9"
+					(reference "R33")
 					(unit 1)
 				)
@@
 		(dnp no)
 		(fields_autoplaced yes)
-		(property "Reference" "R45"
+		(property "Reference" "R48"
 			(at 142.24 115.5699 0)
 			(effects
@@
 			(project "multi-band-equalizer"
 				(path "/a5803ad9-a9e5-4a2c-ab35-f101ba189524/45ab872a-c810-43fb-b03d-ad8b0d23cb6b"
-					(reference "R45")
-					(unit 1)
-				)
-				(path "/a5803ad9-a9e5-4a2c-ab35-f101ba189524/838129ab-a80a-454e-bedd-d4d19cd21db9"
-					(reference "R34")
+					(reference "R48")
+					(unit 1)
+				)
+				(path "/a5803ad9-a9e5-4a2c-ab35-f101ba189524/838129ab-a80a-454e-bedd-d4d19cd21db9"
+					(reference "R37")
 					(unit 1)
 				)
@@
 		(dnp no)
 		(fields_autoplaced yes)
-		(property "Reference" "R43"
+		(property "Reference" "R46"
 			(at 107.95 87.6299 0)
 			(effects
@@
 			(project "multi-band-equalizer"
 				(path "/a5803ad9-a9e5-4a2c-ab35-f101ba189524/45ab872a-c810-43fb-b03d-ad8b0d23cb6b"
-					(reference "R43")
-					(unit 1)
-				)
-				(path "/a5803ad9-a9e5-4a2c-ab35-f101ba189524/838129ab-a80a-454e-bedd-d4d19cd21db9"
-					(reference "R32")
+					(reference "R46")
+					(unit 1)
+				)
+				(path "/a5803ad9-a9e5-4a2c-ab35-f101ba189524/838129ab-a80a-454e-bedd-d4d19cd21db9"
+					(reference "R35")
 					(unit 1)
 				)
@@
 		(dnp no)
 		(fields_autoplaced yes)
-		(property "Reference" "C48"
+		(property "Reference" "C51"
 			(at 119.38 73.66 90)
 			(effects
@@
 			(project "multi-band-equalizer"
 				(path "/a5803ad9-a9e5-4a2c-ab35-f101ba189524/45ab872a-c810-43fb-b03d-ad8b0d23cb6b"
-					(reference "C48")
-					(unit 1)
-				)
-				(path "/a5803ad9-a9e5-4a2c-ab35-f101ba189524/838129ab-a80a-454e-bedd-d4d19cd21db9"
-					(reference "C44")
+					(reference "C51")
+					(unit 1)
+				)
+				(path "/a5803ad9-a9e5-4a2c-ab35-f101ba189524/838129ab-a80a-454e-bedd-d4d19cd21db9"
+					(reference "C47")
 					(unit 1)
 				)
@@
 		(dnp no)
 		(fields_autoplaced yes)
-		(property "Reference" "R48"
+		(property "Reference" "R51"
 			(at 168.91 130.81 90)
 			(effects
@@
 			(project "multi-band-equalizer"
 				(path "/a5803ad9-a9e5-4a2c-ab35-f101ba189524/45ab872a-c810-43fb-b03d-ad8b0d23cb6b"
-					(reference "R48")
-					(unit 1)
-				)
-				(path "/a5803ad9-a9e5-4a2c-ab35-f101ba189524/838129ab-a80a-454e-bedd-d4d19cd21db9"
-					(reference "R37")
+					(reference "R51")
+					(unit 1)
+				)
+				(path "/a5803ad9-a9e5-4a2c-ab35-f101ba189524/838129ab-a80a-454e-bedd-d4d19cd21db9"
+					(reference "R40")
 					(unit 1)
 				)
@@
 		(dnp no)
 		(fields_autoplaced yes)
-		(property "Reference" "R42"
+		(property "Reference" "R45"
 			(at 68.58 87.6299 0)
 			(effects
@@
 			(project "multi-band-equalizer"
 				(path "/a5803ad9-a9e5-4a2c-ab35-f101ba189524/45ab872a-c810-43fb-b03d-ad8b0d23cb6b"
-					(reference "R42")
-					(unit 1)
-				)
-				(path "/a5803ad9-a9e5-4a2c-ab35-f101ba189524/838129ab-a80a-454e-bedd-d4d19cd21db9"
-					(reference "R31")
+					(reference "R45")
+					(unit 1)
+				)
+				(path "/a5803ad9-a9e5-4a2c-ab35-f101ba189524/838129ab-a80a-454e-bedd-d4d19cd21db9"
+					(reference "R34")
 					(unit 1)
 				)
@@
 		(dnp no)
 		(fields_autoplaced yes)
-		(property "Reference" "R39"
+		(property "Reference" "R42"
 			(at 151.13 54.61 90)
 			(effects
@@
 			(project "multi-band-equalizer"
 				(path "/a5803ad9-a9e5-4a2c-ab35-f101ba189524/45ab872a-c810-43fb-b03d-ad8b0d23cb6b"
-					(reference "R39")
-					(unit 1)
-				)
-				(path "/a5803ad9-a9e5-4a2c-ab35-f101ba189524/838129ab-a80a-454e-bedd-d4d19cd21db9"
-					(reference "R28")
+					(reference "R42")
+					(unit 1)
+				)
+				(path "/a5803ad9-a9e5-4a2c-ab35-f101ba189524/838129ab-a80a-454e-bedd-d4d19cd21db9"
+					(reference "R31")
 					(unit 1)
 				)
@@
 		(on_board yes)
 		(dnp no)
-		(property "Reference" "C50"
+		(property "Reference" "C53"
 			(at 168.91 150.622 90)
 			(effects
@@
 			(project "multi-band-equalizer"
 				(path "/a5803ad9-a9e5-4a2c-ab35-f101ba189524/45ab872a-c810-43fb-b03d-ad8b0d23cb6b"
-					(reference "C50")
-					(unit 1)
-				)
-				(path "/a5803ad9-a9e5-4a2c-ab35-f101ba189524/838129ab-a80a-454e-bedd-d4d19cd21db9"
-					(reference "C46")
+					(reference "C53")
+					(unit 1)
+				)
+				(path "/a5803ad9-a9e5-4a2c-ab35-f101ba189524/838129ab-a80a-454e-bedd-d4d19cd21db9"
+					(reference "C49")
 					(unit 1)
 				)
@@
 		(dnp no)
 		(fields_autoplaced yes)
-		(property "Reference" "R38"
+		(property "Reference" "R41"
 			(at 133.35 52.0699 0)
 			(effects
@@
 			(project "multi-band-equalizer"
 				(path "/a5803ad9-a9e5-4a2c-ab35-f101ba189524/45ab872a-c810-43fb-b03d-ad8b0d23cb6b"
-					(reference "R38")
-					(unit 1)
-				)
-				(path "/a5803ad9-a9e5-4a2c-ab35-f101ba189524/838129ab-a80a-454e-bedd-d4d19cd21db9"
-					(reference "R27")
+					(reference "R41")
+					(unit 1)
+				)
+				(path "/a5803ad9-a9e5-4a2c-ab35-f101ba189524/838129ab-a80a-454e-bedd-d4d19cd21db9"
+					(reference "R30")
 					(unit 1)
 				)
@@
 		(dnp no)
 		(fields_autoplaced yes)
-		(property "Reference" "C47"
+		(property "Reference" "C50"
 			(at 250.19 46.99 90)
 			(effects
@@
 			(project "multi-band-equalizer"
 				(path "/a5803ad9-a9e5-4a2c-ab35-f101ba189524/45ab872a-c810-43fb-b03d-ad8b0d23cb6b"
-					(reference "C47")
-					(unit 1)
-				)
-				(path "/a5803ad9-a9e5-4a2c-ab35-f101ba189524/838129ab-a80a-454e-bedd-d4d19cd21db9"
-					(reference "C43")
+					(reference "C50")
+					(unit 1)
+				)
+				(path "/a5803ad9-a9e5-4a2c-ab35-f101ba189524/838129ab-a80a-454e-bedd-d4d19cd21db9"
+					(reference "C46")
 					(unit 1)
 				)
@@
 		(dnp no)
 		(fields_autoplaced yes)
-		(property "Reference" "C49"
+		(property "Reference" "C52"
 			(at 88.9 87.6299 0)
 			(effects
@@
 			(project "multi-band-equalizer"
 				(path "/a5803ad9-a9e5-4a2c-ab35-f101ba189524/45ab872a-c810-43fb-b03d-ad8b0d23cb6b"
-					(reference "C49")
-					(unit 1)
-				)
-				(path "/a5803ad9-a9e5-4a2c-ab35-f101ba189524/838129ab-a80a-454e-bedd-d4d19cd21db9"
-					(reference "C45")
-					(unit 1)
-				)
+					(reference "C52")
+					(unit 1)
+				)
+				(path "/a5803ad9-a9e5-4a2c-ab35-f101ba189524/838129ab-a80a-454e-bedd-d4d19cd21db9"
+					(reference "C48")
+					(unit 1)
+				)
