File: pcb/multi-band-equalizer/multi-band-equalizer.kicad_pcb (KiCad board)
At the start: 4 copper layers, 270.6 x 203.1 mm, 235 parts, among them J1 TagConnect_TC2030, J2 Barrel_Jack_Switch, J3 Input Audio, J4 Output Audio, Q1 SI2347DS-T1-BE3, SW1 SW_Push, U1 CS4272, U10 NE5532, U2 STM32H7B0VBT6, U3 SPX3819M5-L-3-3, U4 SPX3819M5-L-5-0, U5 NE5532, U6 NE5532, U7 NE5532, U8 NE5532, U9 NE5532, Y1 24 MHz

Commit message: update pcb
Parts:
- removed S1: SF12011F-0202-20R-M-050, Custom_Switches:SF12011F020220RM050
- removed the TP11 at (427.9, 127.0)
- removed the TP9 at (427.9, 120.4)
- added FID4: Fiducial, Fiducial:Fiducial_1mm_Mask3mm, B.Cu at (412.0, 153.7)
- added FID5: Fiducial, Fiducial:Fiducial_1mm_Mask3mm, B.Cu at (181.3, 153.7)
- added FID6: Fiducial, Fiducial:Fiducial_1mm_Mask3mm, B.Cu at (405.8, 277.5)
- added G***: LOGO, LOGO, F.Cu at (380.4, 238.6)
- added J5: Conn_01x06_Socket, Connector_Molex:Molex_PicoBlade_53048-0610_1x06_P1.25mm_Horizontal, B.Cu at (343.7, 277.4)
- added TP13: TestPoint, TestPoint:TestPoint_THTPad_D1.0mm_Drill0.5mm, F.Cu at (194.4, 158.0)
- added TP14: TestPoint, TestPoint:TestPoint_THTPad_D1.0mm_Drill0.5mm, F.Cu at (226.0, 180.2)
- added TP15: TestPoint, TestPoint:TestPoint_THTPad_D1.0mm_Drill0.5mm, F.Cu at (247.7, 166.5)
- added TP16: TestPoint, TestPoint:TestPoint_THTPad_D1.0mm_Drill0.5mm, F.Cu at (285.3, 208.3)
- added TP17: TestPoint, TestPoint:TestPoint_THTPad_D1.0mm_Drill0.5mm, F.Cu at (263.8, 222.1)
- added TP18: TestPoint, TestPoint:TestPoint_THTPad_D1.0mm_Drill0.5mm, F.Cu at (311.8, 221.3)
- added TP19: TestPoint, TestPoint:TestPoint_THTPad_D1.0mm_Drill0.5mm, F.Cu at (235.1, 191.2)
- added TP20: TestPoint, TestPoint:TestPoint_THTPad_D1.0mm_Drill0.5mm, F.Cu at (284.7, 196.1)
- added TP21: TestPoint, TestPoint:TestPoint_THTPad_D1.0mm_Drill0.5mm, F.Cu at (235.4, 223.3)
- added TP22: TestPoint, TestPoint:TestPoint_THTPad_D1.0mm_Drill0.5mm, F.Cu at (287.8, 221.4)
- added TP23: TestPoint, TestPoint:TestPoint_THTPad_D1.0mm_Drill0.5mm, F.Cu at (335.8, 221.6)
- added TP5: TestPoint, TestPoint:TestPoint_THTPad_D1.0mm_Drill0.5mm, F.Cu at (280.6, 206.6)
- added TP6: TestPoint, TestPoint:TestPoint_THTPad_D1.0mm_Drill0.5mm, F.Cu at (280.6, 203.5)
- C35, C36, C37, C38, C39, C40, C41, C42, C43, C44, C45, R19, R20, R21, R22, R23, R24, R25, R26, R27, R28, R29, RV1, RV10, RV11, RV2, RV3, RV4, RV5, RV6, RV7, RV8, RV9: moved to B.Cu
- H1, H2, H3, H4: footprint MountingHole:MountingHole_3.2mm_M3_Pad_Via -> MountingHole:MountingHole_4.3mm_M4_Pad_Via
- TP24: renamed from TP13; moved to B.Cu
- TP25: renamed from TP14; moved to B.Cu
- TP26: renamed from TP15; moved to B.Cu
- TP27: renamed from TP16; moved to B.Cu
- TP28: renamed from TP17; moved to B.Cu
- TP29: renamed from TP18; moved to B.Cu
- TP30: renamed from TP19; moved to B.Cu
- TP31: renamed from TP20; moved to B.Cu
- TP32: renamed from TP21; moved to B.Cu
- TP33: renamed from TP22; moved to B.Cu
- TP34: renamed from TP23; moved to B.Cu
- moved J4 330.0 mm to (169.3, 216.5), turned to 180 degrees
- moved H1 319.5 mm to (175.0, 142.4)
- moved FID1 312.5 mm to (185.1, 150.5)
- moved H3 297.4 mm to (175.3, 284.0)
- moved FID3 292.5 mm to (186.6, 278.9)
- moved TP3 252.3 mm to (229.9, 180.2), turned to 180 degrees
- moved SW1 250.6 mm to (229.9, 171.9), turned to 0 degrees
- moved TP2 247.5 mm to (234.5, 194.2), turned to 180 degrees
- moved FID7 240.3 mm to (257.8, 174.9)
- moved C12 238.8 mm to (240.0, 197.1), turned to -90 degrees
- moved C11 237.0 mm to (240.0, 193.3), turned to 90 degrees
- moved FB1 232.7 mm to (242.3, 195.2), turned to -90 degrees
- moved Y1 232.6 mm to (240.8, 185.7), turned to -90 degrees
- moved C13 231.9 mm to (239.6, 175.5), turned to 90 degrees
- moved C10 230.2 mm to (242.9, 190.6), turned to 180 degrees
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- renumbered C30 to C1, C8 to C10, C9 to C11, C10 to C12, C11 to C13, C12 to C14, C13 to C15, C14 to C16, C15 to C17, C16 to C18, C17 to C19, C31 to C2, C18 to C20, C19 to C21, C20 to C22, C21 to C23, C22 to C24, C23 to C25, C24 to C26, C25 to C27, C26 to C28, C27 to C29, C1 to C3, C28 to C30, C29 to C31, C2 to C4, C3 to C5, C4 to C6, C5 to C7, C6 to C8, C7 to C9, FID4 to FID7, J3 to J2, J2 to J3, TP8 to TP10, TP10 to TP11, TP5 to TP7, TP6 to TP8, TP7 to TP9
Connections:
- TP4 pad 1: /I2C_SCL -> /CODEC_NRST
- U2 pad 38: unconnected-(U2-PE8-Pad38) -> /CODEC_NRST
- U2 pad 42: unconnected-(U2-PE12-Pad42) -> /MCU_LED_STATUS_RED
- U2 pad 45: /MCU_LED_STATUS_RED -> unconnected-(U2-PE15-Pad45)
- U2 pad 46: unconnected-(U2-PB10-Pad46) -> /I2C_SCL
- U2 pad 47: unconnected-(U2-PB11-Pad47) -> /I2C_SDA
- U2 pad 56: /CODEC_NRST -> unconnected-(U2-PD9-Pad56)
- U2 pad 66: /I2C_SDA -> unconnected-(U2-PC9-Pad66)
- U2 pad 67: /I2C_SCL -> unconnected-(U2-PA8-Pad67)
Routing:
- net +3.3V: track 0.00 -> 336.9 mm, vias 0 -> 4
- net /CODEC_AOUT_L: track 0.00 -> 324.5 mm
- net /CODEC_AOUT_R: track 0.00 -> 253.0 mm
- net /VDDA: track 0.00 -> 220.9 mm
- net /ASIGNAL_OUT_R: track 0.00 -> 212.2 mm
- net /ASIGNAL_OUT_L: track 0.00 -> 193.8 mm
- net GND: track 0.00 -> 193.5 mm, vias 0 -> 126
- net /ASIGNAL_IN_R: track 0.00 -> 170.7 mm
- net /ASIGNAL_IN_L: track 0.00 -> 148.1 mm
- net /CTRL_KNB_30_HZ: track 0.00 -> 121.2 mm
- net /CTRL_KNB_60_HZ: track 0.00 -> 110.4 mm
- net /CTRL_KNB_120_HZ: track 0.00 -> 99.7 mm
- net /I2C_SCL: track 0.00 -> 98.1 mm, vias 0 -> 2
- net /CODEC_VCOM: track 0.00 -> 96.0 mm, vias 0 -> 2
- net /I2C_SDA: track 0.00 -> 90.0 mm, vias 0 -> 2
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- added copper zone on F.Cu, net +3.3V
- added copper zone on B.Cu, net +5V
- added copper zone on F.Cu, net +5V
- added copper zone on F.Cu, net GND
- added copper zone on In1.Cu, net GND
- added copper zone on In2.Cu, net GND
Other:
- board size 270.6 x 203.1 mm -> 266.7 x 165.1 mm
- board text added: "Analog Input Buffers"
- board text added: "Analog Output Filters"
- board text added: "Audio Codec"
- board text added: "GND"
- board text added: "MCU"
- board text added: "Power"
- board text added: "SWD"
- board text added: "Single-Ended to Differential Converters"
- board text added: "multi-band-equalizer"

Commit message: stitching vias
Parts:
- moved G*** 4.02 mm to (383.0, 241.6)
- moved TP4 0.24 mm to (280.5, 210.4)
Routing:
- net /ASIGNAL_OUT_R: track 212.2 -> 216.8 mm
- net /CTRL_KNB_3200_HZ: track 46.2 -> 47.8 mm
- net +3.3V: track 336.9 -> 335.5 mm
- net /CTRL_KNB_1600_HZ: track 56.9 -> 57.8 mm
- net GND: track 193.5 -> 193.7 mm, vias 126 -> 250

Commit message: pcb update
Parts:
- removed the G*** at (383.0, 241.6)
- added G***: LOGO, LOGO, F.Cu at (231.3, 163.6)
- added G***: LOGO, LOGO, F.Cu at (382.4, 259.5)
- J2: value Input Audio -> Output Audio
- J4: value Output Audio -> Input Audio
- J5: footprint Connector_Molex:Molex_PicoBlade_53048-0610_1x06_P1.25mm_Horizontal -> Connector_JST:JST_XH_S6B-XH-A_1x06_P2.50mm_Horizontal
- moved J4 203.2 mm to (363.1, 155.4), turned to 90 degrees
- moved FID3 185.5 mm to (370.2, 252.5)
- moved J2 77.1 mm to (395.4, 155.4), turned to 90 degrees
- moved R17 76.1 mm to (402.1, 234.7), turned to 90 degrees
- moved R14 75.9 mm to (402.1, 239.5)
- moved FID5 70.1 mm to (243.3, 186.4), turned to -90 degrees
- moved FID1 68.4 mm to (243.3, 186.4), turned to 90 degrees
- moved H1 67.9 mm to (231.5, 180.0)
- moved J5 59.4 mm to (393.6, 245.2)
- moved R16 53.8 mm to (384.5, 235.9), turned to 0 degrees
- moved R15 48.1 mm to (380.2, 235.9), turned to 180 degrees
- moved H3 47.3 mm to (214.3, 257.3)
- moved FID4 46.2 mm to (379.2, 186.3), turned to 90 degrees
- moved FID2 45.8 mm to (379.2, 186.3), turned to -90 degrees
- moved H2 44.7 mm to (401.5, 186.1)
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Connections:
- J2 pad 2: /ASIGNAL_IN_R -> /ASIGNAL_OUT_R
- J2 pad 3: /ASIGNAL_IN_L -> /ASIGNAL_OUT_L
- J2 pad 5: /ASIGNAL_IN_R -> /ASIGNAL_OUT_R
- J2 pad 6: /ASIGNAL_IN_L -> /ASIGNAL_OUT_L
- J4 pad 2: /ASIGNAL_OUT_R -> /ASIGNAL_IN_R
- J4 pad 3: /ASIGNAL_OUT_L -> /ASIGNAL_IN_L
- J4 pad 5: /ASIGNAL_OUT_R -> /ASIGNAL_IN_R
- J4 pad 6: /ASIGNAL_OUT_L -> /ASIGNAL_IN_L
- J5 pad 1: /CODEC_AOUT_R -> /CODEC_AOUT_L
- J5 pad 2: /CODEC_AOUT_L -> /CODEC_AOUT_R
- J5 pad 3: /ASIGNAL_IN_R -> /ASIGNAL_OUT_R
- J5 pad 4: /ASIGNAL_IN_L -> /ASIGNAL_OUT_L
- J5 pad 5: /ASIGNAL_OUT_R -> /ASIGNAL_IN_R
- J5 pad 6: /ASIGNAL_OUT_L -> /ASIGNAL_IN_L
Routing:
- net /ASIGNAL_OUT_R: track 216.8 -> 116.2 mm
- net /CODEC_AOUT_L: track 324.5 -> 235.1 mm
- net /ASIGNAL_OUT_L: track 193.8 -> 108.2 mm
- net /CODEC_AOUT_R: track 253.0 -> 190.4 mm
- net /I2S_LRCK: track 19.0 -> 49.5 mm, vias 0 -> 2
- net /I2S_SCLK: track 19.2 -> 47.5 mm, vias 0 -> 2
- net /ASIGNAL_IN_L: track 148.1 -> 121.0 mm, vias 0 -> 2
- net /ASIGNAL_IN_R: track 170.7 -> 152.9 mm
- net +3.3V: track 335.5 -> 330.8 mm
- net +9V: track 59.9 -> 57.2 mm
- net Net-(U1-VD): track 8.50 -> 9.70 mm
- net GND: track 193.7 -> 193.5 mm, vias 250 -> 214
Other:
- board size 266.7 x 165.1 mm -> 236.9 x 135.2 mm
- board text added: "9VDC / 650mA"
- board text added: "Audio In"
- board text added: "Audio Out"
- board text added: "Footswitch Connector"
