File: pcb/multi-band-equalizer/multi-band-equalizer.kicad_pcb (KiCad board)
At the start: 4 copper layers, 236.9 x 135.2 mm, 251 parts, among them J1 TagConnect_TC2030, J2 Output Audio, J3 Barrel_Jack_Switch, J4 Input Audio, J5 Conn_01x06_Socket, Q1 SI2347DS-T1-BE3, SW1 SW_Push, U1 CS4272, U10 NE5532, U2 STM32H7B0VBT6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

Commit message: new gerbers
Parts:
- C10, C4, C5, C6, C7, C8, C9: value 100n -> 1u
- C3: value 2u2 -> 10u
- J5: moved to F.Cu
- moved J5 12.5 mm to (381.1, 245.2), turned to 0 degrees
- moved G*** 8.89 mm to (386.1, 267.6)
- moved H3 2.27 mm to (216.1, 255.9)
- moved TP15 1.73 mm to (251.7, 189.3)
- moved TP21 1.49 mm to (237.9, 243.9)
- moved TP16 1.17 mm to (288.1, 229.0)
- moved H4 1.02 mm to (404.8, 250.3)
- moved TP14 0.57 mm to (230.1, 200.7)
Connections:
- J5 pad 1: /CODEC_AOUT_L -> /ASIGNAL_IN_L
- J5 pad 2: /CODEC_AOUT_R -> /ASIGNAL_IN_R
- J5 pad 3: /ASIGNAL_OUT_R -> /ASIGNAL_OUT_L
- J5 pad 4: /ASIGNAL_OUT_L -> /ASIGNAL_OUT_R
- J5 pad 5: /ASIGNAL_IN_R -> /CODEC_AOUT_R
- J5 pad 6: /ASIGNAL_IN_L -> /CODEC_AOUT_L
Routing:
- net GND: vias 214 -> 213
Other:
- board text added: "+3.3V"
- board text added: "+9V"
- board text added: "CODEC_NRST"
- board text added: "CTRL_KNB_120_HZ"
- board text added: "CTRL_KNB_12800_HZ"
- board text added: "CTRL_KNB_1600_HZ"
- board text added: "CTRL_KNB_200_HZ"
- board text added: "CTRL_KNB_30_HZ"
- board text added: "CTRL_KNB_3200_HZ"
- board text added: "CTRL_KNB_400_HZ"
- board text added: "CTRL_KNB_60_HZ"
- board text added: "CTRL_KNB_6400_HZ"
- board text added: "CTRL_KNB_800_HZ"
- board text added: "CTRL_KNB_VOL_LVL"
- board text added: "I2C_SCL"
- board text added: "I2C_SDA"
- board text added: "I2S_LRCK"
- board text added: "I2S_MCLK"
- board text added: "I2S_SCLK"
- board text added: "I2S_SDI"
- board text added: "I2S_SDO"
- board text added: "MCU_NRST"
- board text added: "VDDA"

Commit message: resistor value
Parts:
- R12: value 10K -> 10k
Changed lines of the file:
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@@
 			)
 		)
-		(property "Value" "10K"
+		(property "Value" "10k"
 			(at 0 1.65 0)
 			(layer "F.Fab")
