File: pcb/multi-band-equalizer/multi-band-equalizer.kicad_sch (KiCad schematic)
At the start: 68 parts, among them J1 TagConnect_TC2030, J2 Barrel_Jack_Switch, J3 Left Audio In, J4 Right Audio In, J5 Left Audio Out, J6 Right Audio Out, Q1 SI2347DS-T1-BE3, SW1 SW_Push, U1 CS4272, U2 STM32H7B0VBTx, U3 SPX3819M5-L-3-3, U4 SPX3819M5-L-5-0

Commit message: pcb updates
Parts:
- removed C63: 100n, Capacitor_SMD:C_0805_2012Metric, symbol Device:C
- added C10, C34, C35, C36, C37, C38, C39, C40, C41, C8, C9: 100n, Capacitor_SMD:C_0805_2012Metric, symbol Device:C
- added C19, C78, C79: 2u2, Capacitor_SMD:C_0805_2012Metric, symbol Device:C
- added C27, C30: C, Capacitor_SMD:C_0805_2012Metric, symbol Device:C
- added D1: Zener, symbol Device:D_Zener
- added FB1: 120R, Inductor_SMD:L_0805_2012Metric, symbol Device:FerriteBead
- added R14: 2k2, Resistor_SMD:R_0805_2012Metric, symbol Device:R
- added R16, R17, R18, R19: 1M, Resistor_SMD:R_0805_2012Metric, symbol Device:R
- added R20, R21, R22, R23, R24, R25, R26, R27, R8: 5k1, Resistor_SMD:R_0805_2012Metric, symbol Device:R
- added R6: 22R, Resistor_SMD:R_0805_2012Metric, symbol Device:R
- added RV1, RV2, RV3, RV4, RV5, RV6, RV7, RV8: 5k, symbol Device:R_Potentiometer
- added SW2: SW_Push_DPDT, symbol Switch:SW_Push_DPDT
- added Y1: 50 MHz, symbol Device:Crystal
- renumbered C64 to C1, C1 to C11, C2 to C12, C3 to C13, C7 to C14, C8 to C15, C4 to C16, C5 to C17, C6 to C18, C57 to C2, C9 to C20, C10 to C21, C11 to C22, C12 to C23, C15 to C24, C16 to C25, C17 to C26, C13 to C28, C14 to C29, C58 to C3, C18 to C31, C19 to C32, C20 to C33, C59 to C4, C60 to C5, C61 to C6, C62 to C7, D1 to D2, D2 to D3, D3 to D4, D4 to D5, D5 to D6, D6 to D7, D7 to D8, FB1 to FB2, R9 to R10, R7 to R11, R10 to R12, R11 to R13, R12 to R15, R6 to R7, R8 to R9
Connections:
- net I2S_IN is gone; now on net I2S_SDI: U1.7 (SDIN)
- net I2S_OUT is gone; now on net I2S_SDO: R13.1, U1.6 (SDOUT(M/~{S}))
- net +3.3V: now also C1.1, C2.1, C3.1, C4.1, C5.1, C6.1, C7.1, U2.100 (VDD), U2.11 (VDD), U2.27 (VDD), U2.50 (VDD), U2.6 (VBAT), U2.75 (VDD), C10.1, D1.1 (K), FB1.2; no longer U2.20 (VREF+)
- net ASIGNAL_IN_L: now also R18.1, SW2.3 (C)
- net ASIGNAL_IN_R: now also R16.1, SW2.6 (C)
- net ASIGNAL_OUT_L: now also SW2.2 (B)
- net ASIGNAL_OUT_R: now also SW2.5 (B)
- net CODEC_NRST: now also U2.80 (PC12), R8.1; no longer R11.1, U1.14 (~{RST})
- net GND: now also C1.2, C2.2, C3.2, C4.2, C5.2, C6.2, C7.2, SW1.1, C10.2, C19.2, C27.2, C30.2, C34.2, C35.2, C36.2, C37.2, C38.2, C39.2, C40.2, C41.2, C78.2, C79.2, C8.2, C9.2, D1.2 (A), R14.2, R16.2, R17.2, R18.2, R19.2, RV1.3, RV2.3, RV3.3, RV4.3, RV5.3, RV6.3, RV7.3, RV8.3
- net I2C_SCL: now also U2.92 (PB6)
- net I2C_SDA: now also U2.93 (PB7)
- net I2S_LRCK: now also U2.51 (PB12)
- net I2S_MCLK: now also U2.63 (PC6)
- net I2S_SCLK: now also U2.52 (PB13)
- net MCU_NRST: now also SW1.2
- net MCU_SWCLK: now also U2.76 (PA14)
- net MCU_SWDIO: now also U2.72 (PA13)
- net MCU_SWO: now also U2.89 (PB3)
- net MCU_XTI: now reaches U2.12 (PH0)
- net MCU_XTI: now also C27.1, Y1.2
- net at U2.13 (PH1): now also R6.2
- net VDDA: now reaches U2.21 (VDDA)
- net VDDA: now also U2.20 (VREF+), C8.1, C9.1, FB1.1, RV1.1, RV2.1, RV3.1, RV4.1, RV5.1, RV6.1, RV7.1, RV8.1
- net CTRL_KNB_100_HZ: now reaches U2.28 (PA4)
- net CTRL_KNB_100_HZ: now also C34.1, R20.2
- net CTRL_KNB_200_HZ: now reaches U2.29 (PA5)
- net CTRL_KNB_200_HZ: now also C35.1, R21.2
- net CTRL_KNB_400_HZ: now reaches U2.30 (PA6)
- net CTRL_KNB_400_HZ: now also C36.1, R22.2
- net CTRL_KNB_800_HZ: now reaches U2.31 (PA7)
- net CTRL_KNB_800_HZ: now also C37.1, R23.2
- net CTRL_KNB_1600_HZ: now reaches U2.32 (PC4)
- net CTRL_KNB_1600_HZ: now also C38.1, R24.2
- net CTRL_KNB_3200_HZ: now reaches U2.33 (PC5)
- net CTRL_KNB_3200_HZ: now also C39.1, R25.2
- net CTRL_KNB_6400_HZ: now reaches U2.34 (PB0)
- net CTRL_KNB_6400_HZ: now also C40.1, R26.2
- net CTRL_KNB_VOL_LVL: now reaches U2.35 (PB1)
- net CTRL_KNB_VOL_LVL: now also C41.1, R27.2
- net MCU_LED_STATUS_RED: now reaches U2.45 (PE15)
- net MCU_LED_STATUS_RED: now also D6.2 (A)
- net at U2.48 (VCAP): now also C78.1
- net I2S_SDI: now reaches U2.53 (PB14)
- net I2S_SDO: now reaches U2.54 (PB15)
- net at U2.73 (VCAP): now also C79.1
- net at D6.1 (K): now also R14.1
- new net: R23.1, RV4.2
- new net: R26.1, RV7.2
- new net: R27.1, RV8.2
- new net: R22.1, RV3.2
- new net: R24.1, RV5.2
- new net: R20.1, RV1.2
- new net: R21.1, RV2.2
- new net: R25.1, RV6.2
- new net CODEC_AOUT_L: R19.1, SW2.1 (A)
- new net CODEC_AOUT_R: R17.1, SW2.4 (A)
- new net CODEC_NRST_FILT: C19.1, R11.1, R8.2, U1.14 (~{RST})
- new net MCU_XTO: C30.1, R6.1, Y1.1
Other:
- note added: "Control Knobs"
- note added: "Debouncing Capacitor"
- note added: "External Crystal"
- note added: "External Resistor for Crystal Need to calculate for specific crystal"
- note added: "LRCK = 48 kHz SCLK = 64 * LRCK = 3.072 MHz MCLK = 256 * LRCK = 12.288 MHz"
- note added: "Low ESR VCAP Capacitors (<100 mOhms)"
- note added: "MCU Reset Switch"
- note added: "Pull Down Resistors for Anti-Popping"
- note added: "True Bypass"
- note added: "f(-3dB) = 1/(2πRC) = 312 Hz"
- moved on the sheet: C1, C11, C14, C15, C16, C2, C28, C29, C3, C4, C5, C6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

Commit message: Update schematic
Parts:
- removed R6: 22R, Resistor_SMD:R_0805_2012Metric, symbol Device:R
- added TP1: TestPoint, TestPoint:TestPoint_THTPad_D2.0mm_Drill1.0mm, symbol Connector:TestPoint
- Y1: value 50 MHz -> 24 MHz
Connections:
- net MCU_XTO: now also U2.13 (PH1)
Other:
- note removed: "External Resistor for Crystal Need to calculate for specific crystal"
Changed lines of the file:
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@@
 	(wire
 		(pts
-			(xy 406.4 182.88) (xy 408.94 182.88)
-		)
-		(stroke
-			(width 0)
-			(type default)
-		)
-	)
-	(wire
-		(pts
 			(xy 438.15 55.88) (xy 438.15 57.15)
 		)
@@
 	(wire
 		(pts
-			(xy 388.62 180.34) (xy 408.94 180.34)
-		)
-		(stroke
-			(width 0)
-			(type default)
-		)
-	)
-	(wire
-		(pts
 			(xy 288.29 347.98) (xy 316.23 347.98)
 		)
@@
 	(wire
 		(pts
+			(xy 408.94 180.34) (xy 389.89 180.34)
+		)
+		(stroke
+			(width 0)
+			(type default)
+		)
+	)
+	(wire
+		(pts
 			(xy 214.63 340.36) (xy 201.93 340.36)
 		)
@@
 	(wire
 		(pts
+			(xy 408.94 182.88) (xy 389.89 182.88)
+		)
+		(stroke
+			(width 0)
+			(type default)
+		)
+	)
+	(wire
+		(pts
 			(xy 283.21 374.65) (xy 287.02 374.65)
 		)
@@
 	(wire
 		(pts
-			(xy 388.62 182.88) (xy 398.78 182.88)
-		)
-		(stroke
-			(width 0)
-			(type default)
-		)
-	)
-	(wire
-		(pts
 			(xy 161.29 200.66) (xy 119.38 200.66)
 		)
@@
 		)
 	)
-	(text "External Resistor for Crystal\nNeed to calculate for specific crystal"
-		(exclude_from_sim no)
-		(at 381 186.69 0)
-		(effects
-			(font
-				(size 1.27 1.27)
-			)
-		)
-	)
 	(text "Upper 6 bits of the 7 bit address field is always 001000. \nSince we pulled AD0 to VA the chip address will be 0010001\n(Pg 36)"
 		(exclude_from_sim no)
@@
 	)
 	(label "MCU_XTO"
-		(at 388.62 182.88 0)
+		(at 389.89 182.88 0)
 		(fields_autoplaced yes)
 		(effects
@@
 	)
 	(label "MCU_XTI"
-		(at 388.62 180.34 0)
+		(at 389.89 180.34 0)
 		(fields_autoplaced yes)
 		(effects
@@
 	(symbol
 		(lib_id "Device:R")
-		(at 402.59 182.88 90)
-		(unit 1)
-		(exclude_from_sim no)
-		(in_bom yes)
-		(on_board yes)
-		(dnp no)
-		(property "Reference" "R6"
-			(at 402.59 185.42 90)
-			(effects
-				(font
-					(size 1.27 1.27)
-				)
-			)
-		)
-		(property "Value" "22R"
-			(at 402.59 187.96 90)
-			(effects
-				(font
-					(size 1.27 1.27)
-				)
-			)
-		)
-		(property "Footprint" "Resistor_SMD:R_0805_2012Metric"
-			(at 402.59 184.658 90)
-			(effects
-				(font
-					(size 1.27 1.27)
-				)
-				(hide yes)
-			)
-		)
-		(property "Datasheet" "~"
-			(at 402.59 182.88 0)
-			(effects
-				(font
-					(size 1.27 1.27)
-				)
-				(hide yes)
-			)
-		)
-		(property "Description" "Resistor"
-			(at 402.59 182.88 0)
-			(effects
-				(font
-					(size 1.27 1.27)
-				)
-				(hide yes)
-			)
-		)
-		(pin "2"
-		)
-		(pin "1"
-		)
-		(instances
-			(project "multi-band-equalizer"
-				(path "/a5803ad9-a9e5-4a2c-ab35-f101ba189524"
-					(reference "R6")
-					(unit 1)
-				)
-			)
-		)
-	)
-	(symbol
-		(lib_id "Device:R")
 		(at 124.46 213.36 0)
 		(unit 1)
@@
 			)
 		)
-		(property "Value" "50 MHz"
+		(property "Value" "24 MHz"
 			(at 574.04 353.0599 90)
 			(effects
@@
 					(unit 1)
 				)
+			)
+		)
+	)
+	(symbol
+		(lib_id "Connector:TestPoint")
+		(at 595.63 177.8 0)
+		(unit 1)
+		(exclude_from_sim no)
+		(in_bom yes)
+		(on_board yes)
+		(dnp no)
+		(fields_autoplaced yes)
+		(property "Reference" "TP1"
+			(at 598.17 173.2279 0)
+			(effects
+				(font
+					(size 1.27 1.27)
+				)
+				(justify left)
+			)
+		)
+		(property "Value" "TestPoint"
+			(at 598.17 175.7679 0)
+			(effects
+				(font
+					(size 1.27 1.27)
+				)
+				(justify left)
+			)
+		)
+		(property "Footprint" "TestPoint:TestPoint_THTPad_D2.0mm_Drill1.0mm"
+			(at 600.71 177.8 0)
+			(effects
+				(font
+					(size 1.27 1.27)
+				)
+				(hide yes)
+			)
+		)
+		(property "Datasheet" "~"
+			(at 600.71 177.8 0)
+			(effects
+				(font
+					(size 1.27 1.27)
+				)
+				(hide yes)
+			)
+		)
+		(property "Description" "test point"
+			(at 595.63 177.8 0)
+			(effects
+				(font
+					(size 1.27 1.27)
+				)
+				(hide yes)
+			)
+		)
+		(pin "1"
+		)
+		(instances
+			(project ""
+				(path "/a5803ad9-a9e5-4a2c-ab35-f101ba189524"
+					(reference "TP1")
+					(unit 1)
+				)

Commit message: sliding potentiometers
Parts:
- removed RV1, RV2, RV3, RV4, RV5, RV6, RV7: 5k, symbol Device:R_Potentiometer
- added D9: LED_GREEN, LED_SMD:LED_0805_2012Metric, symbol Device:LED
- added R19: 2k2, Resistor_SMD:R_0805_2012Metric, symbol Device:R
- added RV1, RV2, RV3, RV4, RV5, RV6, RV7: 5k, Custom_Potentiometers:PTA2043-2015CPB502, symbol Custom_Potentiometers:PTA2043-2015CPB502
- C10, C9: value 100n -> 2u2
- renumbered C78 to C24, C79 to C25, C24 to C26, C25 to C27, C26 to C28, C27 to C29, C28 to C30, C29 to C31, C30 to C32, C31 to C33, C32 to C34, C33 to C35, C34 to C36, C35 to C37, C36 to C38, C37 to C39, C38 to C40, C39 to C41, C40 to C42, C41 to C43, R11 to R10, R14 to R11, R15 to R14, R16 to R15, R17 to R16, R18 to R17, R19 to R18, R7 to R6, R8 to R7, R9 to R8, R10 to R9
Connections:
- net +5V: now also D9.2 (A)
- net CODEC_NRST: now also U2.69 (PA10); no longer U2.80 (PC12)
- net GND: now also R19.2, RV1.3, RV2.3, RV3.3, RV4.3, RV5.3, RV6.3, RV7.3
- net I2C_SCL: now also U2.67 (PA8); no longer U2.92 (PB6)
- net I2C_SDA: now also U2.66 (PC9); no longer U2.93 (PB7)
- net VDDA: now also RV1.1, RV2.1, RV3.1, RV4.1, RV5.1, RV6.1, RV7.1
- net at R23.1: now also RV4.2
- net at R26.1: now also RV7.2
- net at R22.1: now also RV3.2
- net at R24.1: now also RV5.2
- net at R20.1: now also RV1.2
- net at R21.1: now also RV2.2
- net at R25.1: now also RV6.2
- new net: D9.1 (K), R19.1
- no-connect marks 4 -> 64
Other:
- note added: "f(-3dB) = 1/(2πRC) = 602 Hz"
- note added: "f(-3dB) = 1/(2π√(LC)) = 100 Hz"

Commit message: Update pcb
Parts:
- removed C16, C29, C32: C, Capacitor_SMD:C_0805_2012Metric, symbol Device:C
- removed R18: 1M, Resistor_SMD:R_0805_2012Metric, symbol Device:R
- removed R5: R, Resistor_SMD:R_0805_2012Metric, symbol Device:R
- removed SW2: SW_Push_DPDT, symbol Switch:SW_Push_DPDT
- removed Y1: 24 MHz, symbol Device:Crystal
- added C30, C31: 10p, Capacitor_SMD:C_0805_2012Metric, symbol Device:C
- added R14: 1M, Resistor_SMD:R_0805_2012Metric, symbol Device:R
- added S1: SF12011F-0202-20R-M-050, Custom_Switches:SF12011F020220RM050, symbol Custom_Switches:SF12011F-0202-20R-M-050
- added TP10, TP11, TP12, TP13, TP14, TP15, TP16, TP17, TP18, TP19, TP2, TP20, TP3, TP4, TP5, TP6, TP7, TP8, TP9: TestPoint, TestPoint:TestPoint_THTPad_D1.0mm_Drill0.5mm, symbol Connector:TestPoint
- added Y1: 24 MHz, Crystal:Crystal_SMD_2520-4Pin_2.5x2.0mm, symbol Device:Crystal_GND24
- D1, D2, D3, D4, D5: footprint (none) -> Diode_SMD:D_SOD-323
- SW1: footprint (none) -> Button_Switch_THT:SW_PUSH_6mm_H4.3mm
- TP1: footprint TestPoint:TestPoint_THTPad_D2.0mm_Drill1.0mm -> TestPoint:TestPoint_THTPad_D1.0mm_Drill0.5mm
- renumbered C17 to C16, C18 to C17, C19 to C18, C20 to C19, C21 to C20, C22 to C21, C23 to C22, C24 to C23, C25 to C24, C26 to C25, C27 to C26, C28 to C27, C30 to C28, C31 to C29, C33 to C32, C34 to C33, C35 to C34, C36 to C35, C37 to C36, C38 to C37, C39 to C38, C40 to C39, C41 to C40, C42 to C41, C43 to C42, R11 to R10, R12 to R11, R13 to R12, R14 to R13, R19 to R18, R20 to R19, R21 to R20, R22 to R21, R23 to R22, R24 to R23, R25 to R24, R26 to R25, R27 to R26, R6 to R5, R7 to R6, R8 to R7, R9 to R8, R10 to R9
Connections:
- net +3.3V: now also TP1.1
- net +9V: now also TP12.1
- net ASIGNAL_IN_L: now also R15.1, S1.3 (NC_1); no longer R17.1
- net ASIGNAL_IN_R: now also R16.1, S1.6 (NC_2); no longer R15.1
- net ASIGNAL_OUT_L: now also S1.2 (COM_1)
- net ASIGNAL_OUT_R: now also S1.5 (COM_2)
- net CODEC_AOUT_L: now also R14.1, S1.1 (NO_1)
- net CODEC_AOUT_R: now also R17.1, S1.4 (NO_2); no longer R16.1
- net CODEC_NRST: now also TP5.1
- net CTRL_KNB_100_HZ: now also TP13.1
- net CTRL_KNB_1600_HZ: now also TP17.1
- net CTRL_KNB_200_HZ: now also TP14.1
- net CTRL_KNB_3200_HZ: now also TP18.1
- net CTRL_KNB_400_HZ: now also TP15.1
- net CTRL_KNB_6400_HZ: now also TP19.1
- net CTRL_KNB_800_HZ: now also TP16.1
- net CTRL_KNB_VOL_LVL: now also TP20.1
- net GND: now also C30.2, C31.2, R14.2, Y1.2, Y1.4
- net I2C_SCL: now also TP4.1
- net I2C_SDA: now also TP11.1
- net I2S_LRCK: now also TP6.1
- net I2S_MCLK: now also TP10.1
- net I2S_SCLK: now also TP7.1
- net I2S_SDI: now also TP8.1
- net I2S_SDO: now also TP9.1
- net MCU_NRST: now also TP3.1
- net MCU_XTI: now also C30.1, Y1.1
- net MCU_XTO: now also C31.1, Y1.3
- net VDDA: now also TP2.1
Other:
- note added: "Bypass Switch (DPDT Foot Switch)"
- note added: "CL (Load Capacitance) = 10 pF CS (Stray Capacitance) = ~3-5 pF Effective Load Capacitance = 2(CL-CS) = 2(10-5) = 10 pF"
- note removed: "Bypass Switch"
- note removed: "f(-3dB) = 1/(2π√(LC)) = 100 Hz"

Commit message: Updated pcb and script
Parts:
- removed C42: 100n, Capacitor_SMD:C_0805_2012Metric, symbol Device:C
- removed R26: 5k1, Resistor_SMD:R_0805_2012Metric, symbol Device:R
- removed RV8: 5k, symbol Device:R_Potentiometer
- removed TP20, TP5: TestPoint, TestPoint:TestPoint_THTPad_D1.0mm_Drill0.5mm, symbol Connector:TestPoint
- added C36, C37, C44, C45: 100n, Capacitor_SMD:C_0805_2012Metric, symbol Device:C
- added R20, R21, R28, R29: 5k1, Resistor_SMD:R_0805_2012Metric, symbol Device:R
- added RV10, RV11, RV2, RV3: 5k, Custom_Potentiometers:PTA2043-2015CPB502, symbol Custom_Potentiometers:PTA2043-2015CPB502
- added TP14, TP15, TP22, TP23, TP9: TestPoint, TestPoint:TestPoint_THTPad_D1.0mm_Drill0.5mm, symbol Connector:TestPoint
- C14: value 100n -> 1u
- C15: value 1u -> 100n
- renumbered C36 to C38, C37 to C39, C38 to C40, C39 to C41, C40 to C42, C41 to C43, R20 to R22, R21 to R23, R22 to R24, R23 to R25, R24 to R26, R25 to R27, RV2 to RV4, RV3 to RV5, RV4 to RV6, RV5 to RV7, RV6 to RV8, RV7 to RV9, TP14 to TP16, TP15 to TP17, TP16 to TP18, TP17 to TP19, TP18 to TP20, TP19 to TP21, TP6 to TP5, TP7 to TP6, TP8 to TP7, TP9 to TP8
Connections:
- net CODEC_NRST: now also U2.56 (PD9), TP9.1; no longer U2.69 (PA10)
- net CTRL_KNB_1600_HZ: now also U2.29 (PA5); no longer U2.32 (PC4)
- net CTRL_KNB_200_HZ: now also U2.32 (PC4); no longer U2.29 (PA5)
- net CTRL_KNB_3200_HZ: now also U2.28 (PA4); no longer U2.33 (PC5)
- net CTRL_KNB_400_HZ: now also U2.31 (PA7); no longer U2.30 (PA6)
- net CTRL_KNB_6400_HZ: now also U2.25 (PA3); no longer U2.34 (PB0)
- net CTRL_KNB_800_HZ: now also U2.30 (PA6); no longer U2.31 (PA7)
- net CTRL_KNB_VOL_LVL: now also U2.23 (PA1), C45.1, R29.2, TP23.1; no longer U2.35 (PB1)
- net GND: now also C36.2, C37.2, C44.2, C45.2, RV10.3, RV11.3, RV2.3, RV3.3
- net VDDA: now also RV10.1, RV11.1, RV2.1, RV3.1
- net CTRL_KNB_12800_HZ: now reaches U2.24 (PA2)
- net CTRL_KNB_12800_HZ: now also C44.1, R28.2, TP22.1
- net CTRL_KNB_100_HZ renamed CTRL_KNB_30_HZ
- net CTRL_KNB_30_HZ: now also U2.35 (PB1); no longer U2.28 (PA4)
- new net: R21.1, RV3.2
- new net: R20.1, RV2.2
- new net: R29.1, RV11.2
- new net: R28.1, RV10.2
- new net CTRL_KNB_120_HZ: C37.1, R21.2, TP15.1, U2.33 (PC5)
- new net CTRL_KNB_60_HZ: C36.1, R20.2, TP14.1, U2.34 (PB0)
- no-connect marks 64 -> 61
Other:
- moved on the sheet: C1, C10, C11, C12, C13, C16, C17, C18, C19, C2, C20, C21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

Commit message: update pcb
Parts:
- removed J3: Left Audio In, Connector_Audio:Jack_6.35mm_Neutrik_NJ2FD-V_Vertical, symbol Connector_Audio:AudioJack2
- removed J4: Right Audio In, Connector_Audio:Jack_6.35mm_Neutrik_NJ2FD-V_Vertical, symbol Connector_Audio:AudioJack2
- removed J5: Left Audio Out, Connector_Audio:Jack_6.35mm_Neutrik_NJ2FD-V_Vertical, symbol Connector_Audio:AudioJack2
- removed J6: Right Audio Out, Connector_Audio:Jack_6.35mm_Neutrik_NJ2FD-V_Vertical, symbol Connector_Audio:AudioJack2
- added J3: Input Audio, Custom_Connectors:ACJSMHDR, symbol Custom_Connectors:ACJS-MHDR
- added J4: Output Audio, Custom_Connectors:ACJSMHDR, symbol Custom_Connectors:ACJS-MHDR
- U2: value STM32H7B0VBTx -> STM32H7B0VBT6
Connections:
- net ASIGNAL_IN_L: now also J3.3 (T), J3.6 (T)
- net ASIGNAL_IN_R: now also J3.2 (R), J3.5 (R)
- net ASIGNAL_OUT_L: now also J4.3 (T), J4.6 (T)
- net ASIGNAL_OUT_R: now also J4.2 (R), J4.5 (R)
- net GND: now also J3.1 (S), J3.4 (S), J4.1 (S), J4.4 (S)
Other:
- note added: "1/4 Inch TRS Audio Connections"
- note removed: "All I/O are DNP 1/4 Inch TS Connections"
- moved on the sheet: C30, C31, Y1

Commit message: update pcb
Parts:
- removed TP11, TP9: TestPoint, TestPoint:TestPoint_THTPad_D1.0mm_Drill0.5mm, symbol Connector:TestPoint
- added FID4, FID5, FID6: Fiducial, Fiducial:Fiducial_1mm_Mask3mm, symbol Mechanical:Fiducial
- added J5: Conn_01x06_Socket, Connector_Molex:Molex_PicoBlade_53048-0610_1x06_P1.25mm_Horizontal, symbol Connector:Conn_01x06_Socket
- added TP13, TP14, TP15, TP16, TP17, TP18, TP19, TP20, TP21, TP22, TP23, TP5, TP6: TestPoint, TestPoint:TestPoint_THTPad_D1.0mm_Drill0.5mm, symbol Connector:TestPoint
- H1, H2, H3, H4: footprint MountingHole:MountingHole_3.2mm_M3_Pad_Via -> MountingHole:MountingHole_4.3mm_M4_Pad_Via
- renumbered C30 to C1, C8 to C10, C9 to C11, C10 to C12, C11 to C13, C12 to C14, C13 to C15, C14 to C16, C15 to C17, C16 to C18, C17 to C19, C31 to C2, C18 to C20, C19 to C21, C20 to C22, C21 to C23, C22 to C24, C23 to C25, C24 to C26, C25 to C27, C26 to C28, C27 to C29, C1 to C3, C28 to C30, C29 to C31, C2 to C4, C3 to C5, C4 to C6, C5 to C7, C6 to C8, C7 to C9, FID4 to FID7, J3 to J2, J2 to J3, TP8 to TP10, TP10 to TP11, TP13 to TP24, TP14 to TP25, TP15 to TP26, TP16 to TP27, TP17 to TP28, TP18 to TP29, TP19 to TP30, TP20 to TP31, TP21 to TP32, TP22 to TP33, TP23 to TP34, TP5 to TP7, TP6 to TP8, TP7 to TP9
Connections:
- net ASIGNAL_IN_L: now also J5.4 (Pin_4)
- net ASIGNAL_IN_R: now also J5.3 (Pin_3)
- net ASIGNAL_OUT_L: now also J5.6 (Pin_6)
- net ASIGNAL_OUT_R: now also J5.5 (Pin_5)
- net CODEC_AOUT_L: now also J5.2 (Pin_2)
- net CODEC_AOUT_R: now also J5.1 (Pin_1)
- net CODEC_NRST: now also TP4.1, U2.38 (PE8); no longer U2.56 (PD9)
- net GND: now also TP13.1, TP14.1, TP15.1, TP16.1, TP17.1, TP18.1, TP19.1, TP20.1, TP21.1, TP22.1, TP23.1
- net I2C_SCL: now also U2.46 (PB10), TP5.1; no longer TP4.1, U2.67 (PA8)
- net I2C_SDA: now also U2.47 (PB11), TP6.1; no longer U2.66 (PC9)
- net MCU_LED_STATUS_RED: now also U2.42 (PE12); no longer U2.45 (PE15)
Other:
- note added: "6 Socket Molex Connector for connecting foot switch"
- note added: "Local grounds for the test points"
- note added: "Test Point Grounds"
- moved on the sheet: C1, C2, C35, C36, C37, C38, C39, C40, C41, C42, C43, C44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

Commit message: pcb update
Parts:
- J2: value Input Audio -> Output Audio
- J4: value Output Audio -> Input Audio
- J5: footprint Connector_Molex:Molex_PicoBlade_53048-0610_1x06_P1.25mm_Horizontal -> Connector_JST:JST_XH_S6B-XH-A_1x06_P2.50mm_Horizontal
Connections:
- net ASIGNAL_IN_L: now also J4.3 (T), J4.6 (T), J5.6 (Pin_6); no longer J2.3 (T), J2.6 (T), J5.4 (Pin_4)
- net ASIGNAL_IN_R: now also J4.2 (R), J4.5 (R), J5.5 (Pin_5); no longer J2.2 (R), J2.5 (R), J5.3 (Pin_3)
- net ASIGNAL_OUT_L: now also J2.3 (T), J2.6 (T), J5.4 (Pin_4); no longer J4.3 (T), J4.6 (T), J5.6 (Pin_6)
- net ASIGNAL_OUT_R: now also J2.2 (R), J2.5 (R), J5.3 (Pin_3); no longer J4.2 (R), J4.5 (R), J5.5 (Pin_5)
- net CODEC_AOUT_L: now also J5.1 (Pin_1); no longer J5.2 (Pin_2)
- net CODEC_AOUT_R: now also J5.2 (Pin_2); no longer J5.1 (Pin_1)
Other:
- note added: "6 Socket Molex Connector for connecting footswitch"
- note removed: "6 Socket Molex Connector for connecting foot switch"
